File: STM32F303VCT6.kicad_sch (KiCad schematic)
At the start: 33 parts, among them SW1 SKRPACE010, U2 GD32F303VCT6, Y1 TAXM8M4RDBCCT2T, Y2 XKXGI-SUA-32.768K

Commit message: 更新原理图
Other:
- added sheet Motor_Comm (Motor_Comm.kicad_sch)
- moved on the sheet: C10, C11, C12, C13, C14, C15, C16, C17, C18, C19, C20, C21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

Commit message: 增加USB,TYPEC转串口esd隔离，
Connections:
- net TIMER2_CH0-PWM1: now reaches U2.31 (PA6)
- net TIMER2_CH1-PWM2: now reaches U2.32 (PA7)
- net TIMER2_CH2-PWM3: now reaches U2.35 (PB0)
- net TIMER2_CH3-PWM4: now reaches U2.36 (PB1)
- net TIMER0_CH0-PWM1: now reaches U2.40 (PE9)
- net TIMER0_CH1-PWM2: now reaches U2.42 (PE11)
- net TIMER0_CH2-PWM3: now reaches U2.44 (PE13)
- net TIMER0_CH3-PWM4: now reaches U2.45 (PE14)
- net USART0_TX: now reaches U2.68 (PA9)
- net USART0_RX: now reaches U2.69 (PA10)
- net RS232_RX renamed MCU_RS232_RX
- net RS232_TX renamed MCU_RS232_TX
Other:
- added sheet USB_TTL_CH340 (TTL_CH340.kicad_sch)
- moved on the sheet: C25, C26, U2E
