File: GD32F303VCT6.kicad_sch (KiCad schematic)
At the start: 32 parts, among them SW1 SKRPACE010, U6 GD32F303VCT6, Y1 TAXM8M4RDBCCT2T, Y2 XKXGI-SUA-32.768K

Commit message: 调整DIR1与DIR2引脚映射并优化局部布局
交换 PD0-PD3 与 PC14、PC15、PC6、PC7 的 DIR1/DIR2 功能分配，同步更新 PCB 网络，并调整 JP2 与 R11 位置。
Connections:
- net DIR1_1: now also U6.81 (PD0); no longer U6.33 (DIR1)
- net DIR1_2: now also U6.82 (PD1); no longer U6.34 (DIR2)
- net DIR1_3: now also U6.83 (PD2); no longer U6.63 (DIR3)
- net DIR1_4: now also U6.84 (PD3); no longer U6.64 (DIR4)
- net DIR2_1: now also U6.33 (DIR1); no longer U6.81 (PD0)
- net DIR2_2: now also U6.34 (DIR2); no longer U6.82 (PD1)
- net DIR2_3: now also U6.63 (DIR3); no longer U6.83 (PD2)
- net DIR2_4: now also U6.64 (DIR4); no longer U6.84 (PD3)
Changed lines of the file:
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@@
 		)
 	)
-	(label "DIR2_1"
+	(label "DIR1_1"
 		(at 335.28 134.62 0)
 		(effects
@@
 		)
 	)
-	(label "DIR2_2"
+	(label "DIR1_2"
 		(at 335.28 138.43 0)
 		(effects
@@
 		)
 	)
-	(label "DIR1_3"
+	(label "DIR2_3"
 		(at 162.56 153.67 0)
 		(effects
@@
 		)
 	)
-	(label "DIR2_[1..4]"
+	(label "DIR1_[1..4]"
 		(at 347.98 130.81 0)
 		(effects
@@
 		)
 	)
-	(label "DIR1_[1..4]"
+	(label "DIR2_[1..4]"
 		(at 175.26 142.24 0)
 		(effects
@@
 		)
 	)
-	(label "DIR1_1"
+	(label "DIR2_1"
 		(at 162.56 146.05 0)
 		(effects
@@
 		)
 	)
-	(label "DIR1_2"
+	(label "DIR2_2"
 		(at 162.56 149.86 0)
 		(effects
@@
 		)
 	)
-	(label "DIR2_4"
+	(label "DIR1_4"
 		(at 335.28 146.05 0)
 		(effects
@@
 		)
 	)
-	(label "DIR2_3"
+	(label "DIR1_3"
 		(at 335.28 142.24 0)
 		(effects
@@
 		)
 	)
-	(label "DIR1_4"
+	(label "DIR2_4"
 		(at 162.56 157.48 0)
 		(effects

Commit message: 完善总线映射并划分隔离地与电源平面
统一3V3电源网络并消除ERC错误；优化GND/Earth耦合器件布局；完成In1.Cu地平面及In2.Cu电源平面分区。
Connections:
- net BRAKE1_1: now also U6.81 (PD0); no longer U6.85 (BRAKE1)
- net BRAKE1_2: now also U6.83 (PD2); no longer U6.86 (BRAKE2)
- net BRAKE1_3: now also U6.85 (BRAKE1); no longer U6.87 (BRAKE3)
- net BRAKE1_4: now also U6.87 (BRAKE3); no longer U6.88 (BRAKE4)
- net BRAKE2_1: now also U6.53 (PB14); no longer U6.89 (PB3)
- net BRAKE2_2: now also U6.54 (PB15); no longer U6.90 (PB4)
- net BRAKE2_3: now also U6.55 (PD8); no longer U6.91 (PB5)
- net BRAKE2_4: now also U6.56 (PD9); no longer U6.92 (PB6)
- net DIR1_1: now also U6.82 (PD1); no longer U6.81 (PD0)
- net DIR1_2: now also U6.84 (PD3); no longer U6.82 (PD1)
- net DIR1_3: now also U6.86 (BRAKE2); no longer U6.83 (PD2)
- net DIR1_4: now also U6.88 (BRAKE4); no longer U6.84 (PD3)
- net DIR2_3: now also U6.51 (PB12); no longer U6.63 (DIR3)
- net DIR2_4: now also U6.52 (PB13); no longer U6.64 (DIR4)
- net +3.3V renamed +3V3
- net USB_DM renamed USB_DN
Other:
- sheet USB_TTL_CH340 ports: added USB_DN; removed USB_DM
