File: GD32F303VCT6.kicad_sch (KiCad schematic)
At the start: 32 parts, among them SW1 SKRPACE010, U6 GD32F303VCT6, Y1 TAXM8M4RDBCCT2T, Y2 XKXGI-SUA-32.768K

Commit message: 更新PCB层叠铺铜与器件封装配置
Connections:
- net GND: now also C21.2; no longer C21.1
- net at D5.3, U6.6 (VBAT): now also C21.1; no longer C21.2
Other:
- moved on the sheet: C21
Changed lines of the file:
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@@
 	(symbol
 		(lib_id "Device:C")
-		(at 36.83 48.26 90)
+		(at 36.83 48.26 270)
+		(mirror x)
 		(unit 1)
 		(body_style 1)
@@
 		(in_pos_files yes)
 		(dnp no)
-		(fields_autoplaced yes)
 		(property "Reference" "C21"
 			(at 36.83 40.64 90)
@@
 		)
 		(property "Footprint" "Capacitor_SMD:C_0603_1608Metric"
-			(at 40.64 47.2948 0)
+			(at 33.02 47.2948 0)
 			(hide yes)
 			(show_name no)
@@
 		(exclude_from_sim no)
 		(in_bom yes)
-		(on_board yes)
-		(in_pos_files yes)
-		(dnp no)
+		(on_board no)
+		(in_pos_files no)
+		(dnp yes)
 		(fields_autoplaced yes)
 		(property "Reference" "#PWR043"
