File: GD32F303.kicad_pcb (KiCad board)
At the start: 4 copper layers, 100 x 60 mm, 126 parts, among them CN1 KF128L-5.08-2P, CN2 WJ15EDGRC-3.81-2P, CN4 WJ15EDGRC-3.81-2P, J1 TYPE-C-31-M-31, J2 TYPE-C 16PIN 2MD(073), Q1 CJ3134K KF, Q2 CJ3134K KF, SW1 SKRPACE010, U1 XL1509-5.0, U10 SIT3485ESA, U11 TXS0104EPWR, U12 TXS0104EPWR, U13 CH340E, U14 TPD4S012DRYR, U2 B0503S-2WR3L, U3 SY8089A1AAC, U4 CH213K, U5 SY8089AAC, U6 GD32F303VCT6, U7 ISO1050DWR, U9 π131U30, Y1 TAXM8M4RDBCCT2T, Y2 XKXGI-SUA-32.768K

Commit message: 更新PCB层叠铺铜与器件封装配置
Parts:
- moved C15 0.50 mm to (142.8, 86.7)
- moved Y1 0.50 mm to (142.7, 83.7)
- moved C20 0.33 mm to (142.8, 80.4)
- moved L4 0.31 mm to (96.5, 72.1)
- moved J1 0.30 mm to (92.2, 74.5)
- moved CN4 0.05 mm to (170.4, 62.0)
- turned C52 to 180 degrees
Connections:
- C21 pad 1: GND -> Net-(U6A-VBAT)
- C21 pad 2: Net-(U6A-VBAT) -> GND
Routing:
- net GND: track 132.6 -> 301.2 mm, vias 23 -> 180
- net +5V: track 72.3 -> 155.4 mm, vias 1 -> 4
- net GNDS: track 57.2 -> 124.5 mm, vias 5 -> 22
- net +5V_ISO: track 20.9 -> 85.2 mm, vias 3 -> 8
- net +3V3: track 85.3 -> 129.7 mm, vias 19 -> 25
- net Earth: track 262.8 -> 280.1 mm
- net +3V3_ISO: track 18.2 -> 28.6 mm, vias 0 -> 2
- net /RS485/RS485_TX: track 6.87 -> 8.55 mm
- net /MCU_Core/USB_TTL_CH340/DN: track 8.04 -> 9.67 mm
- net /MCU_Core/FG1_1: track 48.5 -> 50.0 mm
- net Net-(U6A-VBAT): track 10.7 -> 11.9 mm
- net /RS485/RS485_RX: track 9.12 -> 10.0 mm
- net /MCU_Core/RS485_TX: track 49.5 -> 50.3 mm
- net /RS485/CTRL: track 6.81 -> 7.33 mm
- net /MCU_Core/OSCOUT: track 11.5 -> 12.0 mm
- added copper zone on B.Cu, net Earth
- added copper zone on B.Cu, net GND
- added copper zone on F.Cu, net GND
- added copper zone on B.Cu, net GNDS
- added copper zone on F.Cu, net GNDS
Other:
- board text added: "+24V"
- board text added: "+3V3"
- board text added: "BOOT0"
- board text added: "BOOT1"
- board text added: "BRK1_1"
- board text added: "BRK1_2"
- board text added: "BRK1_3"
- board text added: "BRK1_4"
- board text added: "BRK2_1"
- board text added: "BRK2_2"
- board text added: "BRK2_3"
- board text added: "BRK2_4"
- board text added: "CANH"
- board text added: "CANL"
- board text added: "CH340"
- board text added: "CLK"
- board text added: "DIO"
- board text added: "DIR1_1"
- board text added: "DIR1_2"
- board text added: "DIR1_3"
- board text added: "DIR1_4"
- board text added: "DIR2_1"
- board text added: "DIR2_2"
- board text added: "DIR2_3"
- board text added: "DIR2_4"
- board text added: "FG1_1"
- board text added: "FG1_2"
- board text added: "FG1_3"
- board text added: "FG1_4"
- board text added: "FG2_1"
- board text added: "FG2_2"
- board text added: "FG2_3"
- board text added: "FG2_4"
- board text added: "GND"
- board text added: "PWM1_1"
- board text added: "PWM1_2"
- board text added: "PWM1_3"
- board text added: "PWM1_4"
- board text added: "PWM2_1"
- board text added: "PWM2_2"
- board text added: "PWM2_3"
- board text added: "PWM2_4"
- board text added: "RS485A"
- board text added: "RS485B"
- board text added: "RST"
- board text added: "USB"
