File: TTL_CH340.kicad_sch (KiCad schematic)
At the start: 30 parts, among them J1 TYPE-C-31-M-31, J2 TYPE-C 16PIN 2MD(073), Q1 CJ3134K KF, Q2 CJ3134K KF, U13 CH340E, U15 TPD4S012DRYR

Commit message: 完成GD32F303控制板原理图与PCB设计
- 更新电源、CAN、RS232、RS485及电机通信子电路
- 切换并完善GD32F303VCT6核心原理图
- 新增PCB布局及所需符号、封装库文件
Parts:
- C49: renamed from C52; footprint kicad_community_lib:C1005X5R1H104K050BB -> Capacitor_SMD:C_0402_1005Metric_Pad0.74x0.62mm_HandSolder
- C50: renamed from C53; footprint kicad_api_lib:C1005X5R1H104K050BB -> Capacitor_SMD:C_0402_1005Metric_Pad0.74x0.62mm_HandSolder
- C51: renamed from C54; footprint kicad_api_lib:CC1206MKX7RDBB102 -> Capacitor_SMD:C_1206_3216Metric_Pad1.33x1.80mm_HandSolder
- C52: renamed from C55; footprint kicad_api_lib:0603X106M100NT -> Capacitor_SMD:C_0603_1608Metric_Pad1.08x0.95mm_HandSolder
- C53: renamed from C56; footprint kicad_api_lib:C1005X5R1H104K050BB -> Capacitor_SMD:C_0402_1005Metric_Pad0.74x0.62mm_HandSolder
- FB2: footprint kicad_api_lib:UPZ1608E101-3R0TF -> Capacitor_SMD:C_0603_1608Metric_Pad1.08x0.95mm_HandSolder
- J1: footprint kicad_api_lib:TYPE-C-31-M-31 -> kicad_api_lib:TYPE-C 16PIN 2MD(073)
- L4: footprint kicad_api_lib:PCAQ2012B-900T040 -> Inductor_SMD:L_CommonModeChoke_Coilcraft_0805USB
- Q1, Q2: footprint kicad_api_lib:CJ3134K KF -> Package_TO_SOT_SMD:SOT-23-3
- R19: renamed from R17; footprint kicad_api_lib:RC0603JR-130RL -> Resistor_SMD:R_0603_1608Metric_Pad0.98x0.95mm_HandSolder
- R20: renamed from R22; footprint kicad_community_lib:RC0603JR-130RL -> Resistor_SMD:R_0603_1608Metric_Pad0.98x0.95mm_HandSolder
- R21: renamed from R23; footprint kicad_api_lib:RC0603JR-130RL -> Resistor_SMD:R_0603_1608Metric_Pad0.98x0.95mm_HandSolder
- R22: renamed from R24; footprint kicad_community_lib:RTT02472JTH -> Resistor_SMD:R_0402_1005Metric_Pad0.72x0.64mm_HandSolder
- R23: renamed from R25; footprint kicad_api_lib:RC0603JR-130RL -> Resistor_SMD:R_0603_1608Metric_Pad0.98x0.95mm_HandSolder
- R24: renamed from R26; footprint kicad_community_lib:RTT02472JTH -> Resistor_SMD:R_0402_1005Metric_Pad0.72x0.64mm_HandSolder
- R25: renamed from R27; footprint kicad_api_lib:RC0603JR-130RL -> Resistor_SMD:R_0603_1608Metric_Pad0.98x0.95mm_HandSolder
- R26: renamed from R28; footprint kicad_api_lib:RC0402FR-075K1L -> Resistor_SMD:R_0402_1005Metric_Pad0.72x0.64mm_HandSolder
- R27: renamed from R29; footprint kicad_api_lib:RC0402FR-075K1L -> Resistor_SMD:R_0402_1005Metric_Pad0.72x0.64mm_HandSolder
- R28: renamed from R30; footprint kicad_community_lib:RTT02472JTH -> Resistor_SMD:R_0402_1005Metric_Pad0.72x0.64mm_HandSolder
- R29: renamed from R31; footprint kicad_community_lib:RTT02472JTH -> Resistor_SMD:R_0402_1005Metric_Pad0.72x0.64mm_HandSolder
- R30: renamed from R8; footprint kicad_api_lib:0402WGF220JTCE -> Resistor_SMD:R_0402_1005Metric_Pad0.72x0.64mm_HandSolder
- R31: renamed from R15; footprint kicad_api_lib:0402WGF220JTCE -> Resistor_SMD:R_0402_1005Metric_Pad0.72x0.64mm_HandSolder
- R32, R33: footprint kicad_api_lib:0402WGF5101TCE -> Resistor_SMD:R_0402_1005Metric_Pad0.72x0.64mm_HandSolder
- U14: renamed from U15; footprint kicad_api_lib:TPD4S012DRYR -> Package_DFN_QFN:TPD4S012DRYR
- renumbered D8 to D7, D7 to D8

Commit message: 优化接口原理图与PCB布局
- 精简CAN接口并调整各子页器件编号
- 更新电源输入端子与Type-C接口封装
- 重新整理控制板PCB器件布局
Parts:
- J1, J2: footprint kicad_api_lib:TYPE-C 16PIN 2MD(073) -> kicad_api_lib:TYPE-C 16PIN 2MD NEW(073)
Changed lines of the file:
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@@
 			)
 		)
-		(property "Footprint" "kicad_api_lib:TYPE-C 16PIN 2MD(073)"
+		(property "Footprint" "kicad_api_lib:TYPE-C 16PIN 2MD NEW(073)"
 			(at 189.23 52.07 0)
 			(hide yes)
@@
 			)
 		)
-		(property "Footprint" "kicad_api_lib:TYPE-C 16PIN 2MD(073)"
+		(property "Footprint" "kicad_api_lib:TYPE-C 16PIN 2MD NEW(073)"
 			(at 335.28 139.7 0)
 			(hide yes)

Commit message: 完善PCB布线与接口电源网络
- 调整控制板PCB器件布局与走线
- 更新MCU、电源及通信接口原理图
- 统一隔离接口地和电源网络标签并修正封装属性
Parts:
- R19, R21: now left out of the parts list
Connections:
- net CH_RX: now also U13.8 (TXD); no longer R25.2, U13.9 (RXD)
- net CH_TX: now also R25.2, U13.9 (RXD); no longer U13.8 (TXD)

Commit message: 完善总线映射并划分隔离地与电源平面
统一3V3电源网络并消除ERC错误；优化GND/Earth耦合器件布局；完成In1.Cu地平面及In2.Cu电源平面分区。
Connections:
- net USB_DM renamed USB_DN
Changed lines of the file:
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@@
 		)
 	)
-	(hierarchical_label "USB_DM"
+	(hierarchical_label "USB_DN"
 		(shape bidirectional)
 		(at 279.4 121.92 180)

Commit message: 更新六层控制板设计及嘉立创生产文件
Parts:
- renumbered C49 to C50, C50 to C51, C51 to C52, C52 to C53, C53 to C54, D8 to D10, D7 to D9, Q1 to Q3, Q2 to Q4, R19 to R21, R20 to R22, R21 to R23, R22 to R24, R23 to R25, R24 to R26, R25 to R27, R26 to R28, R27 to R29, R28 to R30, R29 to R31, R30 to R32, R31 to R33, R32 to R34, R33 to R35

Commit message: 更新六层电机控制板设计与器件库
Connections:
- net CH_RX: now also R27.2, U13.9 (RXD); no longer U13.8 (TXD)
- net CH_TX: now also U13.8 (TXD); no longer R27.2, U13.9 (RXD)
Changed lines of the file:
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@@
 		)
 	)
-	(label "CH_TX"
+	(label "CH_RX"
 		(at 123.19 68.58 180)
 		(effects
@@
 		)
 	)
-	(label "CH_RX"
+	(label "CH_TX"
 		(at 123.19 66.04 180)
 		(effects
@@
 		(dnp no)
 		(fields_autoplaced yes)
-		(property "Reference" "#FLG013"
+		(property "Reference" "#FLG014"
 			(at 58.42 64.135 0)
 			(hide yes)
@@
 			(project "GD32F303VET6_4Motor_Control"
 				(path "/54005433-e3aa-4693-8f75-bb73943288d3/ab5b236f-20a8-4993-b87c-2c1c522e6f92/1b78379e-163c-4192-b7b2-c6b42c88e9cb"
-					(reference "#FLG013")
+					(reference "#FLG014")
 					(unit 1)
 				)

Commit message: 更新电源与USB供电设计、PCB及器件库
Parts:
- removed R27: 0, Resistor_SMD:R_0603_1608Metric_Pad0.98x0.95mm_HandSolder, symbol RC0603JR-130RL:RC0603JR-130RL
- added C55, C56: 1uF/10V, Capacitor_SMD:C_0603_1608Metric, symbol Device:C
- added U16, U17: LM66100DCKR, kicad_api_lib:LM66100DCKR, symbol kicad_api_lib:LM66100DCKR
- C53: value 10uF -> 4.7uF
- renumbered R28 to R27, R29 to R28, R30 to R29, R31 to R30, R32 to R31, R33 to R32, R34 to R33, R35 to R34
Connections:
- net +5V: now also U16.3 (CE#), U16.6 (VOUT), U17.3 (CE#), U17.6 (VOUT); no longer C53.1, C54.1, J1.A4 (VBUS), J1.A9 (VBUS), J1.B4 (VBUS), J1.B9 (VBUS), J2.A4 (VBUS), J2.A9 (VBUS), J2.B4 (VBUS), J2.B9 (VBUS), U14.6 (VBUS)
- net GND: now also C55.2, C56.2, U16.2 (GND), U16.5 (ST), U17.2 (GND), U17.5 (ST)
- new net USB1_VBUS: C53.1, C54.1, C55.1, J1.A4 (VBUS), J1.A9 (VBUS), J1.B4 (VBUS), J1.B9 (VBUS), U14.6 (VBUS), U16.1 (VIN)
- new net USB2_VBUS: C56.1, J2.A4 (VBUS), J2.A9 (VBUS), J2.B4 (VBUS), J2.B9 (VBUS), U17.1 (VIN)
- no-connect marks 9 -> 12
