File: TTL_CH340.kicad_sch (KiCad schematic)
At the start: 33 parts, among them J1 TYPE-C-31-M-31, J2 TYPE-C 16PIN 2MD(073), Q3 CJ3134K KF, Q4 CJ3134K KF, U13 CH340E, U14 TPD4S012DRYR, U16 LM66100DCKR, U17 LM66100DCKR

Commit message: V2.0: sync KiCad design, add firmware snapshot and README
Parts:
- removed R25: 0, Resistor_SMD:R_0603_1608Metric_Pad0.98x0.95mm_HandSolder, symbol RC0603JR-130RL:RC0603JR-130RL
- added C58: 1uF, Capacitor_SMD:C_0603_1608Metric, symbol Project_Passives:CL10A105KA8NNNC_5d127244
- added C59: 100nF, Capacitor_SMD:C_0603_1608Metric, symbol Project_Passives:CL10B104KB8NNNC_3cb423e4
- added D18, D19: KLXES15AAA1, kicad_api_lib:KLXES15AAA1, symbol KLXES15AAA1:KLXES15AAA1
- added L5: PCAQ2012B-900T040, kicad_api_lib:PCAQ2012B-900T040, symbol PCAQ2012B-900T040:PCAQ2012B-900T040
- added U19: CH340N, kicad_api_lib:CH340N, symbol CH340N:CH340N
- C55: renamed from C50; footprint Capacitor_SMD:C_0402_1005Metric_Pad0.74x0.62mm_HandSolder -> Capacitor_SMD:C_0603_1608Metric; symbol C1005X5R1H104K050BB:C1005X5R1H104K050BB -> Project_Passives:CL10B104KB8NNNC_4873395a; Capacitance 100 nF -> 100nF; Composition Ceramic -> (none); Dielectric (none) -> X7R; Dielectric Material Ceramic -> (none); Height 500 µm -> (none); Lead Free Lead Free -> (none); Length 1 mm -> (none); MPN (none) -> CL10B104KB8NNNC; Manufacturer TDK -> Samsung Electro-Mechanics; Mount Surface Mount -> (none); Mpn C1005X5R1H104K050BB -> (none); Operating Temperature 85 °C -> (none); REACH SHVC Compliant No SVHC -> (none); Temperature Characteristic X5R -> (none); Termination SMD -> (none); Tolerance 10 % -> 10%; Voltage Rating 50 V -> (none); Voltage_Rating (none) -> 50V; Width 0.02 in -> (none); package (none) -> 0603; now not fitted; now left out of the parts list
- C56: renamed from C51; footprint Capacitor_SMD:C_0402_1005Metric_Pad0.74x0.62mm_HandSolder -> Capacitor_SMD:C_0603_1608Metric; symbol C1005X5R1H104K050BB:C1005X5R1H104K050BB -> Project_Passives:CL10B104KB8NNNC_4873395a; Capacitance (none) -> 100nF; Dielectric (none) -> X7R; MPN C1005X5R1H104K050BB -> CL10B104KB8NNNC; Manufacturer TDK -> Samsung Electro-Mechanics; Tolerance (none) -> 10%; Voltage_Rating (none) -> 50V; application General Purpose -> (none); body_length 1 mm -> (none); body_width 0.02 in -> (none); capacitance 100 nF -> (none); case_code_imperial 0402 -> (none); characteristic Low ESL -> (none); composition Ceramic -> (none); depth 500 µm -> (none); dielectric_material Ceramic -> (none); grade 通用级 -> (none); height 500 µm -> (none); huaqiu_pn G0030431 -> (none); lead_free Lead Free -> (none); mount Surface Mount -> (none); operating_temperature -55 °C, 85 °C -> (none); package 0402 -> 0603; package_quantity 1 -> (none); packaging Tape and Reel -> (none); radiation_hardening No -> (none); reach_svhc_compliant No SVHC -> (none); temperature_characteristic X5R -> (none); terminal_pitch 0.90 mm -> (none); termination SMD -> (none); thickness 0.022 in -> (none); tolerance 10 % -> (none); voltage 50 V -> (none); voltage_rating 50 V -> (none); now not fitted; now left out of the parts list
- C57: renamed from C55; footprint Capacitor_SMD:C_0603_1608Metric -> Capacitor_SMD:C_0402_1005Metric
- C60: renamed from C52; value 1nF -> CC1206MKX7RDBB102; footprint Capacitor_SMD:C_1206_3216Metric_Pad1.33x1.80mm_HandSolder -> kicad_api_lib:CC1206MKX7RDBB102
- C62: renamed from C53; value 4.7uF -> 0603X106M100NT; footprint Capacitor_SMD:C_0603_1608Metric_Pad1.08x0.95mm_HandSolder -> Capacitor_SMD:C_0603_1608Metric
- C63: renamed from C54; value 100nF -> C1005X5R1H104K050BB; footprint Capacitor_SMD:C_0402_1005Metric_Pad0.74x0.62mm_HandSolder -> Capacitor_SMD:C_0402_1005Metric
- FB2: value 100ohm@100MHz -> UPZ1608E101-3R0TF; footprint Capacitor_SMD:C_0603_1608Metric_Pad1.08x0.95mm_HandSolder -> kicad_api_lib:UPZ1608E101-3R0TF
- J1, J2: footprint kicad_api_lib:TYPE-C 16PIN 2MD NEW(073) -> kicad_api_lib:TYPE-C-31-M-31
- L4: footprint Inductor_SMD:L_CommonModeChoke_Coilcraft_0805USB -> kicad_api_lib:PCAQ2012B-900T040; now not fitted; now left out of the parts list
- Q16: renamed from Q3; footprint Package_TO_SOT_SMD:SOT-23-3 -> kicad_api_lib:CJ3134K KF
- Q17: renamed from Q4; footprint Package_TO_SOT_SMD:SOT-23-3 -> kicad_api_lib:CJ3134K KF
- R66: renamed from R21; footprint Resistor_SMD:R_0603_1608Metric_Pad0.98x0.95mm_HandSolder -> Resistor_SMD:R_0402_1005Metric; symbol RC0603JR-130RL:RC0603JR-130RL -> Project_Passives:RC0402JR-070RL_f7672f5a; MPN RC0603JR-130RL -> RC0402JR-070RL; Manufacturer Yageo -> YAGEO; Power (none) -> 0.063W; Resistance (none) -> 0; body_length 1.6 mm -> (none); body_width 0.8 mm -> (none); case_code_imperial 0603 -> (none); characteristic Moisture Resistant -> (none); composition Thick Film -> (none); contact_plating Tin -> (none); depth 800 µm -> (none); height 450 µm -> (none); height_overall 0.45 mm -> (none); huaqiu_pn G6239406 -> (none); lead_free Lead Free -> (none); material Thick Film -> (none); military_standard Not -> (none); mount SMT -> (none); operating_temperature -55 °C -> (none); overload_voltage 75 V -> (none); package 0603 -> 0402; packaging Tape and Reel -> (none); pins 2 -> (none); power_rating 100 mW -> (none); radiation_hardening No -> (none); reach_svhc_compliant No SVHC -> (none); resistance 0 Ω -> (none); temperature_coefficient 200 ppm/°C -> (none); terminal_pitch 1.35 mm -> (none); termination SMD -> (none); tolerance 0.05 -> (none); type 厚膜电阻 -> (none); voltage_rating 50 V -> (none)
- R67: renamed from R22; value 0 -> RC0603JR-130RL; footprint Resistor_SMD:R_0603_1608Metric_Pad0.98x0.95mm_HandSolder -> Resistor_SMD:R_0603_1608Metric; Composition Thick Film -> (none); Height 450 µm -> (none); Lead Free Lead Free -> (none); Length 1.6 mm -> (none); MPN (none) -> RC0603JR-130RL; Material Thick Film -> (none); Military Standard Not -> (none); Mount 表面贴装 -> (none); Mpn RC0603JR-130RL -> (none); Operating Temperature 155 °C -> (none); Operating Temperature (Max) 155 °C -> (none); Operating Temperature (Min) -55 °C -> (none); Pins 2 defualt -> (none); Power Rating 100 mW -> (none); REACH SHVC Compliant No SVHC -> (none); Resistance 0 Ω -> (none); Temperature Coefficient 200 ppm/°C -> (none); Termination SMD -> (none); Tolerance 5 % -> (none); Voltage Rating 50 V -> (none); Width 800 µm -> (none); body_length (none) -> 1.6 mm; body_width (none) -> 0.8 mm; case_code_imperial (none) -> 0603; characteristic (none) -> Moisture Resistant; composition (none) -> Thick Film; contact_plating (none) -> Tin; depth (none) -> 800 µm; height (none) -> 450 µm; height_overall (none) -> 0.45 mm; huaqiu_pn (none) -> G6239406; lead_free (none) -> Lead Free; material (none) -> Thick Film; military_standard (none) -> Not; mount (none) -> SMT; operating_temperature (none) -> -55 °C; overload_voltage (none) -> 75 V; package (none) -> 0603; packaging (none) -> Tape and Reel; pins (none) -> 2; power_rating (none) -> 100 mW; radiation_hardening (none) -> No; reach_svhc_compliant (none) -> No SVHC; resistance (none) -> 0 Ω; temperature_coefficient (none) -> 200 ppm/°C; terminal_pitch (none) -> 1.35 mm; termination (none) -> SMD; tolerance (none) -> 0.05; type (none) -> 厚膜电阻; voltage_rating (none) -> 50 V; now not fitted; now left out of the parts list
- R68: renamed from R23; footprint Resistor_SMD:R_0603_1608Metric_Pad0.98x0.95mm_HandSolder -> Resistor_SMD:R_0402_1005Metric; symbol RC0603JR-130RL:RC0603JR-130RL -> Project_Passives:RC0402JR-070RL_f7672f5a; MPN RC0603JR-130RL -> RC0402JR-070RL; Manufacturer Yageo -> YAGEO; Power (none) -> 0.063W; Resistance (none) -> 0; body_length 1.6 mm -> (none); body_width 0.8 mm -> (none); case_code_imperial 0603 -> (none); characteristic Moisture Resistant -> (none); composition Thick Film -> (none); contact_plating Tin -> (none); depth 800 µm -> (none); height 450 µm -> (none); height_overall 0.45 mm -> (none); huaqiu_pn G6239406 -> (none); lead_free Lead Free -> (none); material Thick Film -> (none); military_standard Not -> (none); mount SMT -> (none); operating_temperature -55 °C -> (none); overload_voltage 75 V -> (none); package 0603 -> 0402; packaging Tape and Reel -> (none); pins 2 -> (none); power_rating 100 mW -> (none); radiation_hardening No -> (none); reach_svhc_compliant No SVHC -> (none); resistance 0 Ω -> (none); temperature_coefficient 200 ppm/°C -> (none); terminal_pitch 1.35 mm -> (none); termination SMD -> (none); tolerance 0.05 -> (none); type 厚膜电阻 -> (none); voltage_rating 50 V -> (none)
- R69: renamed from R24; value 4.7K -> 4.7k; footprint Resistor_SMD:R_0402_1005Metric_Pad0.72x0.64mm_HandSolder -> Resistor_SMD:R_0603_1608Metric; symbol RTT02472JTH:RTT02472JTH -> Project_Passives:RC0603JR-074K7L_d4074a4b; Lead Free Yes -> (none); MPN (none) -> RC0603JR-074K7L; Manufacturer Ralec -> YAGEO; Material 金属陶瓷 -> (none); Mount 表面贴装 -> (none); Mpn RTT02472JTH -> (none); Operating Temperature 155 °C -> (none); Operating Temperature (Max) 155 °C -> (none); Operating Temperature (Min) -55 °C -> (none); Power (none) -> 0.1W; Power Rating 62.5 mW -> (none); Resistance (none) -> 4.7k; Technology 厚膜 -> (none); Temperature Coefficient 100 ppm/°C -> (none); Tolerance 5 % -> 5%; package (none) -> 0603
- R70: renamed from R26; value 4.7K -> 4.7k; footprint Resistor_SMD:R_0402_1005Metric_Pad0.72x0.64mm_HandSolder -> Resistor_SMD:R_0603_1608Metric; symbol RTT02472JTH:RTT02472JTH -> Project_Passives:RC0603JR-074K7L_d4074a4b; Lead Free Yes -> (none); MPN (none) -> RC0603JR-074K7L; Manufacturer Ralec -> YAGEO; Material 金属陶瓷 -> (none); Mount 表面贴装 -> (none); Mpn RTT02472JTH -> (none); Operating Temperature 155 °C -> (none); Operating Temperature (Max) 155 °C -> (none); Operating Temperature (Min) -55 °C -> (none); Power (none) -> 0.1W; Power Rating 62.5 mW -> (none); Resistance (none) -> 4.7k; Technology 厚膜 -> (none); Temperature Coefficient 100 ppm/°C -> (none); Tolerance 5 % -> 5%; package (none) -> 0603
- R71: renamed from R27; value 5.1K -> RC0402FR-075K1L; footprint Resistor_SMD:R_0402_1005Metric_Pad0.72x0.64mm_HandSolder -> Resistor_SMD:R_0402_1005Metric
- R72: renamed from R28; value 5.1K -> RC0402FR-075K1L; footprint Resistor_SMD:R_0402_1005Metric_Pad0.72x0.64mm_HandSolder -> Resistor_SMD:R_0402_1005Metric
- R73: renamed from R29; value 4.7K -> 4.7k; footprint Resistor_SMD:R_0402_1005Metric_Pad0.72x0.64mm_HandSolder -> Resistor_SMD:R_0603_1608Metric; symbol RTT02472JTH:RTT02472JTH -> Project_Passives:RC0603JR-074K7L_d4074a4b; Lead Free Yes -> (none); MPN (none) -> RC0603JR-074K7L; Manufacturer Ralec -> YAGEO; Material 金属陶瓷 -> (none); Mount 表面贴装 -> (none); Mpn RTT02472JTH -> (none); Operating Temperature 155 °C -> (none); Operating Temperature (Max) 155 °C -> (none); Operating Temperature (Min) -55 °C -> (none); Power (none) -> 0.1W; Power Rating 62.5 mW -> (none); Resistance (none) -> 4.7k; Technology 厚膜 -> (none); Temperature Coefficient 100 ppm/°C -> (none); Tolerance 5 % -> 5%; package (none) -> 0603
- R74: renamed from R30; value 4.7K -> 4.7k; footprint Resistor_SMD:R_0402_1005Metric_Pad0.72x0.64mm_HandSolder -> Resistor_SMD:R_0603_1608Metric; symbol RTT02472JTH:RTT02472JTH -> Project_Passives:RC0603JR-074K7L_d4074a4b; Lead Free Yes -> (none); MPN (none) -> RC0603JR-074K7L; Manufacturer Ralec -> YAGEO; Material 金属陶瓷 -> (none); Mount 表面贴装 -> (none); Mpn RTT02472JTH -> (none); Operating Temperature 155 °C -> (none); Operating Temperature (Max) 155 °C -> (none); Operating Temperature (Min) -55 °C -> (none); Power (none) -> 0.1W; Power Rating 62.5 mW -> (none); Resistance (none) -> 4.7k; Technology 厚膜 -> (none); Temperature Coefficient 100 ppm/°C -> (none); Tolerance 5 % -> 5%; package (none) -> 0603
- R75: renamed from R31; value 22 -> 0402WGF220JTCE; footprint Resistor_SMD:R_0402_1005Metric_Pad0.72x0.64mm_HandSolder -> Resistor_SMD:R_0402_1005Metric
- R76: renamed from R32; value 22 -> 0402WGF220JTCE; footprint Resistor_SMD:R_0402_1005Metric_Pad0.72x0.64mm_HandSolder -> Resistor_SMD:R_0402_1005Metric
- R77: renamed from R33; value 5.1K -> 0402WGF5101TCE; footprint Resistor_SMD:R_0402_1005Metric_Pad0.72x0.64mm_HandSolder -> Resistor_SMD:R_0402_1005Metric
- R78: renamed from R34; value 5.1K -> 0402WGF5101TCE; footprint Resistor_SMD:R_0402_1005Metric_Pad0.72x0.64mm_HandSolder -> Resistor_SMD:R_0402_1005Metric
- U17: renamed from U13; now not fitted; now left out of the parts list
- U18: renamed from U14; footprint Package_DFN_QFN:TPD4S012DRYR -> kicad_api_lib:TPD4S012DRYR; now not fitted; now left out of the parts list
- U20: renamed from U16; fet_type (none) -> P通道; huaqiu_pn (none) -> G4607254; lead_free (none) -> Yes; mount (none) -> SMT; package (none) -> SC-70-6; packaging (none) -> 3000pcs; voltage (none) -> 1.5 V
- U21: renamed from U17; fet_type (none) -> P通道; huaqiu_pn (none) -> G4607254; lead_free (none) -> Yes; mount (none) -> SMT; package (none) -> SC-70-6; packaging (none) -> 3000pcs; voltage (none) -> 1.5 V
- renumbered C56 to C61, D9 to D20, D10 to D21
Connections:
- net +5V: now also C58.1, U19.5 (VCC)
- net CH_RX: now also U19.7 (RXD); no longer U17.9 (RXD)
- net CH_TX: now also U19.6 (TXD); no longer U17.8 (TXD)
- net DN: now also L5.1
- net DP: now also L5.4
- net Earth: now also D20.1 (A1), D21.2 (A2), J2.MH1, J2.MH2, J2.MH3, J2.MH4
- net GND: now also C58.2, C59.2, D18.1, D19.1, U19.3 (GND); no longer D20.1 (A1), D21.2 (A2), J2.MH1, J2.MH2, J2.MH3, J2.MH4
- new net: D18.2, L5.3, U19.1 (UD+)
- new net: D19.2, L5.2, U19.2 (UD-)
- new net: C59.1, U19.8 (V3)
- no-connect marks 12 -> 15
Other:
- note added: "CH_TX → Q17 → USART0_RX。 R73 / R74 为两侧上拉。"
- note added: "FB2 / C60 Earth ↔ GND"
- note added: "J1 → DP / DN → USB-02；VBUS → USB-06。 R71 / R72：CC 下拉；C62 / C63：VBUS 滤波。"
- note added: "J2 → USB_DP / USB_DN → MCU。 R75 / R76：串阻；D20 / D21：ESD 防护。 R77 / R78：CC 下拉；VBUS → USB-07。"
- note added: "L5：共模滤波；D18 / D19：ESD 防护。 U19：USB 转 UART；C58 / C59：电源去耦。"
- note added: "U17 / L4 / R66~R68 / C55 / C56。 保留原连接作为备选；当前不装配。"
- note added: "U18：TPD4S012DRYR。 当前不装配。"
- note added: "USART0_TX → Q16 → CH_RX。 +3V3 / +5V 共地转换；不构成电气隔离。"
- note added: "USB-01 USB1 / 串口入口"
- note added: "USB-02 CH340N 串口桥"
- note added: "USB-03 MCU 原生 USB 接口"
- note added: "USB-04 UART 发送电平转换"
- note added: "USB-05 UART 接收电平转换"
- note added: "USB-06 USB1 防倒灌供电"
- note added: "USB-07 USB2 防倒灌供电"
- note added: "USB-08 机壳与信号地耦合"
- note added: "USB-09 CH340E 历史备选【备用 / DNP】"
- note added: "USB-10 集成防护芯片备选【备用 / DNP】"
- note added: "USB1_VBUS → U20 → +5V；C57 旁路。"
- note added: "USB2_VBUS → U21 → +5V；C61 旁路。"
- note added: "USB｜串口桥、MCU USB 与供电支路"
- note added: "接口说明 USB1 用于 CH340N 串口桥；USB2 连接 MCU USB。 两个接口的 5 V 电源经各自 U20 / U21 汇入 +5V。 +5V 同时接入 POWER 页 U5 的板内电源支路。 CC 下拉用于 Type-C 受电端识别；当前没有 PD 协议控制器。 USB 信号地接 GND，金属外壳接 Earth。 MOS UART 电平转换为共地电路，速度需按实测边沿确认。 DNP 分区保留原图；“备用”不代表该方案已完成电气验证。"
- note removed: "33-->5V"
- note removed: "33<--5V"
- note removed: "340端"
- note removed: "CH340E_USB TO UART Module"
- note removed: "CH340供电可用板内电源，与处理器电源保持一致； CH340 USB电源如果和处理器IO电源不一致，需要考虑串口倒灌问题；"
- note removed: "TYPE-C 16PIN 2MD(073)_Type-C Connector Module"
- note removed: "UART 电平转换 电源域隔离"
- note removed: "处理器端"
- note removed: "模块电路功能： CH340E是一款 USB 转串口芯片，支持完整的异步串行通信功能，波特率范围通常在 50bps 到 2Mbps 之间。 通过适当的电平转换还可支持 RS232、RS485 和 RS422 接口标准。工作电压通常为 3.3V 或 5V。 该原理图带有完整的接口防护以及电平转化电路。"
- note removed: "模块电路功能： 这是一个符合 USB-IF 规范的基础款 USB 2.0 Type-C 从设备接口电路，完整支持 USB PD 快充， 核心实现Type-C 正反插兼容、USB 2.0 高速数据传输、5V 设备供电、ESD 静电防护四大核心功能。 应用场景： 该电路广泛应用于仅需基础供电 + USB 数据功能的设备，例如：嵌入式开发板 / 核心板、智能家居设备等。"
- moved on the sheet: C57, C60, C61, C62, C63, D20, D21, FB2, J1, J2, Q16, Q17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

Commit message: V2.0: update motor control schematics, replicated PCB layout and component libraries
Save current KiCad design progress, including four motor control layouts and new component libraries. PCB routing and DRC cleanup remain unfinished; this is not a fabrication release.
Parts:
- C62: footprint Capacitor_SMD:C_0603_1608Metric -> Capacitor_SMD:C_0402_1005Metric
Connections:
- net DN: now also L5.3; no longer L5.1
- net DP: now also L5.2; no longer L5.4
- net at D18.2, U19.1 (UD+): now also L5.1; no longer L5.3
- net at D19.2, U19.2 (UD-): now also L5.4; no longer L5.2

Commit message: 更新V2.0电路设计及0.5oz内层制造交付资料
Parts:
- removed D20, D21: SD03C, kicad_api_lib:SD03C, symbol SD03C:TVS-2
- removed R77, R78: 0402WGF5101TCE, Resistor_SMD:R_0402_1005Metric, symbol 0402WGF5101TCE:0402WGF5101TCE
- added D20: PRTR5V0U2X, kicad_api_lib:PRTR5V0U2X, symbol PRTR5V0U2X:PRTR5V0U2X
- added R65: 0402WGF1001TCE, kicad_api_lib:0402WGF1001TCE, symbol 0402WGF1001TCE:R_US
- added TP_CH_RX1: CH_RX, kicad_api_lib:TestPoint_Pad_D0.762mm, symbol Connector:TestPoint
- added TP_CH_TX1: CH_TX, kicad_api_lib:TestPoint_Pad_D0.762mm, symbol Connector:TestPoint
- added TP_GND_USB1: GND_USB, kicad_api_lib:TestPoint_Pad_D1.016mm, symbol Connector:TestPoint
- added TP_MCU_RX1: MCU_RX, kicad_api_lib:TestPoint_Pad_D0.762mm, symbol Connector:TestPoint
- added TP_MCU_TX1: MCU_TX, kicad_api_lib:TestPoint_Pad_D0.762mm, symbol Connector:TestPoint
- added TP_VBUS1: VBUS1, kicad_api_lib:TestPoint_Pad_D1.143mm, symbol Connector:TestPoint
- added TP_VBUS2: VBUS2, kicad_api_lib:TestPoint_Pad_D1.143mm, symbol Connector:TestPoint
- renumbered C55 to C59, C56 to C60, C57 to C61, C58 to C62, C59 to C63, C60 to C64, C61 to C65, C62 to C66, C63 to C67, Q16 to Q4, Q17 to Q5, R66 to R54, R67 to R55, R68 to R56, R69 to R57, R70 to R58, R71 to R59, R72 to R60, R73 to R61, R74 to R62, R75 to R63, R76 to R64, U17 to U21, U18 to U22, U19 to U23, U20 to U24, U21 to U25
Connections:
- net +3V3: now also R65.1
- net CH_RX: now also TP_CH_RX1.1
- net CH_TX: now also TP_CH_TX1.1
- net DN2: now also D20.3 (I/O2)
- net DP2: now also D20.2 (I/O1), R65.2
- net Earth: now also D20.1 (GND)
- net GND: now also TP_GND_USB1.1
- net USB1_VBUS: now also TP_VBUS1.1
- net USB2_VBUS: now also D20.4 (VCC), TP_VBUS2.1
- net USART0_RX renamed USART2_RX
- net USART2_RX: now also TP_MCU_RX1.1
- net USART0_TX renamed USART2_TX
- net USART2_TX: now also TP_MCU_TX1.1
- no-connect marks 15 -> 17
Other:
- note added: "CH_TX → Q5 → USART2_RX / PD9。 R61 / R62 上拉；不构成电气隔离。"
- note added: "J1 → DP / DN → USB-02。 R59 / R60：5.1k CC 下拉；C66 / C67：VBUS 滤波。"
- note added: "J2 → R63 / R64 → PA12 D+ / PA11 D-。 D20：PRTR5V0U2X，当前参考地接 Earth。 R65：D+ 上拉；VBUS 经 U25 接 +5V。 J2 的 CC1 / CC2 当前未连接，需另行复核。"
- note added: "U21 / L4 / R54～R56 / C59、C60。 保留原连接，当前不装配。"
- note added: "U22：TPD4S012DRYR。 当前不装配。"
- note added: "U23：CH340N；L5：共模滤波。 D18 / D19：信号防护；C62 / C63：去耦。"
- note added: "U24：USB1_VBUS → +5V。 C61：输入旁路。"
- note added: "U25：USB2_VBUS → +5V。 C65：输入旁路。"
- note added: "USART2_TX / PD8 → Q4 → CH_RX。 R57 / R58 上拉；3V3 / 5V 共地转换。"
- note added: "USB / UART TEST POINTS"
- note added: "USB-01 USB1 串口入口"
- note added: "USB-03 GD32 原生 USB"
- note added: "USB-04 发送转换"
- note added: "USB-05 接收转换"
- note added: "USB-08 Earth / GND 耦合"
- note added: "USB-09 CH340E 历史备选【DNP】"
- note added: "USB-10 集成 USB 防护备选【DNP】"
- note added: "USB-11 接口说明与待复核项"
- note added: "USB1：CH340N → 电平转换 → GD32 USART2。 USB2：GD32 原生 USB；两路数据通道独立。 USB1 / USB2 / POWER 电源支路汇入 +5V。 接口信号地为 GND，外壳为 Earth。 FB2 / C64：Earth 与 GND 高频耦合。 本次仅整理图纸与新增 PA15 LED，不修改 USB 电路。 J2 的 CC 未接；D20 的回流路径及 R65 取值需另行评估。 旧注释中的元件编号已按当前工程更新。 备用区按实际 DNP / BOM / PCB 属性处理。"
- note added: "USB｜串口桥、MCU USB 与供电"
- note removed: "CH_TX → Q17 → USART0_RX。 R73 / R74 为两侧上拉。"
- note removed: "FB2 / C60 Earth ↔ GND"
- note removed: "J1 → DP / DN → USB-02；VBUS → USB-06。 R71 / R72：CC 下拉；C62 / C63：VBUS 滤波。"
- note removed: "J2 → USB_DP / USB_DN → MCU。 R75 / R76：串阻；D20 / D21：ESD 防护。 R77 / R78：CC 下拉；VBUS → USB-07。"
- note removed: "L5：共模滤波；D18 / D19：ESD 防护。 U19：USB 转 UART；C58 / C59：电源去耦。"
- note removed: "U17 / L4 / R66~R68 / C55 / C56。 保留原连接作为备选；当前不装配。"
- note removed: "U18：TPD4S012DRYR。 当前不装配。"
- note removed: "USART0_TX → Q16 → CH_RX。 +3V3 / +5V 共地转换；不构成电气隔离。"
- note removed: "USB-01 USB1 / 串口入口"
- note removed: "USB-03 MCU 原生 USB 接口"
- note removed: "USB-04 UART 发送电平转换"
- note removed: "USB-05 UART 接收电平转换"
- note removed: "USB-08 机壳与信号地耦合"
- note removed: "USB-09 CH340E 历史备选【备用 / DNP】"
- note removed: "USB-10 集成防护芯片备选【备用 / DNP】"
- note removed: "USB1_VBUS → U20 → +5V；C57 旁路。"
- note removed: "USB2_VBUS → U21 → +5V；C61 旁路。"
- note removed: "USB｜串口桥、MCU USB 与供电支路"
- note removed: "接口说明 USB1 用于 CH340N 串口桥；USB2 连接 MCU USB。 两个接口的 5 V 电源经各自 U20 / U21 汇入 +5V。 +5V 同时接入 POWER 页 U5 的板内电源支路。 CC 下拉用于 Type-C 受电端识别；当前没有 PD 协议控制器。 USB 信号地接 GND，金属外壳接 Earth。 MOS UART 电平转换为共地电路，速度需按实测边沿确认。 DNP 分区保留原图；“备用”不代表该方案已完成电气验证。"
