File: POWER.kicad_sch (KiCad schematic)
At the start: 49 parts, among them CN1 KF128L-5.08-2P, Q1 AP40P04Q, Q2 MMDT5401, U1 XL1509-5.0, U18 LM66100DCKR, U2 IB0505S-2W3L, U3 SY8089A1AAC, U4 CH213K, U5 SY8089AAC

Commit message: V2.0: sync KiCad design, add firmware snapshot and README
Parts:
- added C10, C12: 1nF, Capacitor_SMD:C_0603_1608Metric, symbol Device:C_Small
- added D4: LED, LED_SMD:LED_0603_1608Metric, symbol Device:LED
- added R3: 10kΩ, Resistor_SMD:R_0603_1608Metric, symbol Device:R_US
- added R6, R8: 1MΩ, Resistor_SMD:R_0603_1608Metric, symbol Device:R_US
- C1: value 470µF -> RVT1E471M0810; footprint Capacitor_SMD:CP_Elec_8x10 -> kicad_api_lib:RVT1E471M0810
- C11: footprint Capacitor_SMD:C_0603_1608Metric_Pad1.08x0.95mm_HandSolder -> Capacitor_SMD:C_0603_1608Metric
- C13: renamed from C57; value 4.7uF/10V -> 1uF/10V
- C14: renamed from C9; value 10uF -> 22uF; footprint Capacitor_SMD:C_0603_1608Metric_Pad1.08x0.95mm_HandSolder -> Capacitor_SMD:C_0603_1608Metric; symbol CL10A106MP8NNNC:CL10A106MP8NNNC -> Project_Passives:CL10A226MP8NUNC_bf2966a3; Capacitance (none) -> 22uF; Design_Note (none) -> Verify effective capacitance under DC bias at operating vol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; Dielectric (none) -> X5R; MFG Samsung -> (none); MPN CL10A106MP8NNNC -> CL10A226MP8NUNC; Manufacturer Samsung -> Samsung Electro-Mechanics; Tolerance (none) -> 20%; Voltage_Rating (none) -> 10V; application General Purpose -> (none); body_length 1.6 mm -> (none); body_width 0.031 in -> (none); capacitance 10 μF -> (none); case_code_imperial 0603 -> (none); contact_plating Tin -> (none); depth 800 µm -> (none); dielectric_material 陶瓷 -> (none); grade 通用级 -> (none); height 800 µm -> (none); lead_free Lead Free -> (none); mount Surface Mount -> (none); operating_temperature -55 °C, 85 °C -> (none); package_quantity 1 -> (none); packaging Tape and Reel -> (none); radiation_hardening No -> (none); temperature_characteristic X5R -> (none); terminal_pitch 1.30 mm -> (none); thickness 0.035 in -> (none); tolerance 20 % -> (none); voltage_rating 10 V -> (none)
- C15: renamed from C10; footprint Capacitor_SMD:C_0603_1608Metric_Pad1.08x0.95mm_HandSolder -> Capacitor_SMD:C_0603_1608Metric; symbol 0402B104K500CT:0402B104K500CT -> Project_Passives:CL10B104KB8NNNC_46c1dd14; Capacitance (none) -> 100nF; Dielectric (none) -> X7R; MFG Walsin Technologies -> (none); MPN 0402B104K500CT -> CL10B104KB8NNNC; Manufacturer Walsin Technologies -> Samsung Electro-Mechanics; Tolerance (none) -> 10%; Voltage_Rating (none) -> 50V; grade 消费级 -> (none); lead_free Yes -> (none); mount 表面贴装 -> (none); package 0402 -> 0603; packaging 10000pcs -> (none); tolerance 10 % -> (none); voltage_rating 50 V -> (none)
- C16: renamed from C13; value 100nF -> 22pF; footprint Capacitor_SMD:C_0603_1608Metric_Pad1.08x0.95mm_HandSolder -> Capacitor_SMD:C_0603_1608Metric; symbol 0402B104K500CT:0402B104K500CT -> Project_Passives:CL10C220JB8NNNC_46c1dd14; Capacitance (none) -> 22pF; Dielectric (none) -> C0G; MFG Samsung Electro-Mechanics -> (none); MPN CL10B104KB8NNNC -> CL10C220JB8NNNC; Tolerance (none) -> 5%; Voltage_Rating (none) -> 50V; grade 消费级 -> (none); lead_free Yes -> (none); mount 表面贴装 -> (none); tolerance 10 % -> (none); voltage_rating 50 V -> (none)
- C17: renamed from C14; footprint Capacitor_SMD:C_0603_1608Metric_Pad1.08x0.95mm_HandSolder -> Capacitor_SMD:C_0603_1608Metric; symbol GRM188R61A226ME15D:GRM188R61A226ME15D -> Project_Passives:CL10A226MP8NUNC_53f55199; Capacitance (none) -> 22uF; Design_Note (none) -> Verify effective capacitance under DC bias at operating vol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; Dielectric (none) -> X5R; MFG Murata -> (none); MPN GRM188R61A226ME15D -> CL10A226MP8NUNC; Manufacturer Murata -> Samsung Electro-Mechanics; Tolerance (none) -> 20%; Voltage_Rating (none) -> 10V; application General Purpose -> (none); body_length 1.6 mm -> (none); body_width 0.8 mm -> (none); capacitance 22 μF -> (none); case_code_imperial 0603 -> (none); depth 800 µm -> (none); grade 通用级 -> (none); height 800 µm -> (none); height_overall 0.8 mm -> (none); lead_free Lead Free -> (none); material Ceramic -> (none); mount SMT -> (none); operating_temperature -55 °C -> (none); packaging Tape and Reel -> (none); pins 2 -> (none); reach_svhc_compliant No SVHC -> (none); temperature_characteristic X5R -> (none); termination SMD -> (none); thickness 0.039 in -> (none); tolerance 20 % -> (none); voltage_rating 10 V -> (none); weight 0.000222 oz -> (none)
- C18: renamed from C15; footprint Capacitor_SMD:C_0603_1608Metric_Pad1.08x0.95mm_HandSolder -> Capacitor_SMD:C_0603_1608Metric; symbol 0402B104K500CT:0402B104K500CT -> Project_Passives:CL10B104KB8NNNC_46c1dd14; Capacitance (none) -> 100nF; Dielectric (none) -> X7R; MFG Walsin Technologies -> (none); MPN 0402B104K500CT -> CL10B104KB8NNNC; Manufacturer Walsin Technologies -> Samsung Electro-Mechanics; Tolerance (none) -> 10%; Voltage_Rating (none) -> 50V; grade 消费级 -> (none); lead_free Yes -> (none); mount 表面贴装 -> (none); package 0402 -> 0603; packaging 10000pcs -> (none); tolerance 10 % -> (none); voltage_rating 50 V -> (none)
- C19: renamed from C12; value 100nF -> CC0603KRX7R9BB104; footprint Capacitor_SMD:C_0603_1608Metric_Pad1.08x0.95mm_HandSolder -> Capacitor_SMD:C_0603_1608Metric
- C2: value 10uF -> 22uF; footprint Capacitor_SMD:C_0603_1608Metric_Pad1.08x0.95mm_HandSolder -> Capacitor_SMD:C_0603_1608Metric; symbol Device:C -> Project_Passives:CL10A226MP8NUNC_0447ed23; Capacitance (none) -> 22uF; Design_Note (none) -> Verify effective capacitance under DC bias at operating vol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; Dielectric (none) -> X5R; MPN (none) -> CL10A226MP8NUNC; Manufacturer (none) -> Samsung Electro-Mechanics; Tolerance (none) -> 20%; Voltage_Rating (none) -> 10V; package (none) -> 0603; now not fitted; now left out of the parts list
- C3: value 4.7uF -> C; footprint Capacitor_SMD:C_0603_1608Metric_Pad1.08x0.95mm_HandSolder -> Capacitor_SMD:C_0603_1608Metric; now not fitted; now left out of the parts list
- C4: footprint Capacitor_SMD:C_0603_1608Metric_Pad1.08x0.95mm_HandSolder -> Capacitor_SMD:C_0603_1608Metric; symbol Device:C -> Project_Passives:CL10C220JB8NNNC_0447ed23; Capacitance (none) -> 22pF; Dielectric (none) -> C0G; MPN (none) -> CL10C220JB8NNNC; Manufacturer (none) -> Samsung Electro-Mechanics; Tolerance (none) -> 5%; Voltage_Rating (none) -> 50V; package (none) -> 0603; now not fitted; now left out of the parts list
- C5: value 220µF -> RVT1E221M0607; footprint Capacitor_SMD:CP_Elec_6.3x7.7 -> kicad_api_lib:RVT1E221M0607
- C6: value 10uF -> C; footprint Capacitor_SMD:C_0603_1608Metric_Pad1.08x0.95mm_HandSolder -> Capacitor_SMD:C_0603_1608Metric; now not fitted; now left out of the parts list
- C7: value 10uF -> 22uF; footprint Capacitor_SMD:C_0805_2012Metric_Pad1.18x1.45mm_HandSolder -> Capacitor_SMD:C_0603_1608Metric; symbol Device:C -> Project_Passives:CL10A226MP8NUNC_0447ed23; Capacitance (none) -> 22uF; Design_Note (none) -> Verify effective capacitance under DC bias at operating vol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; Dielectric (none) -> X5R; MPN (none) -> CL10A226MP8NUNC; Manufacturer (none) -> Samsung Electro-Mechanics; Tolerance (none) -> 20%; Voltage_Rating (none) -> 10V; package (none) -> 0603; now not fitted; now left out of the parts list
- C8: value 1uF -> 100nF; footprint Capacitor_SMD:C_0603_1608Metric_Pad1.08x0.95mm_HandSolder -> Capacitor_SMD:C_0603_1608Metric; now not fitted; now left out of the parts list
- D2, D3: footprint LED_SMD:LED_0603_1608Metric_Pad1.05x0.95mm_HandSolder -> LED_SMD:LED_0603_1608Metric
- D6: renamed from D5; footprint Package_TO_SOT_SMD:TSOT-23_HandSoldering -> kicad_api_lib:MMBD1504A
- D7: renamed from D6; footprint Diode_SMD:D_SOD-123 -> kicad_api_lib:BZT52C12
- H1, H2, H3, H4: footprint MountingHole:MountingHole_3.2mm_M3_ISO7380_Pad -> (none)
- L2: renamed from L1; value MWTC201610S1R0MT -> 1uH; now not fitted; now left out of the parts list
- L3: footprint Inductor_SMD_Wurth:L_Wurth_WE-LQSH-3012 -> kicad_api_lib:SWPA3015S2R2NT
- Q2: footprint Package_TO_SOT_SMD:SOT-363_SC-70-6 -> kicad_api_lib:MMDT5401
- R1, R2: value 10k -> 10kΩ; footprint Resistor_SMD:R_0603_1608Metric_Pad0.98x0.95mm_HandSolder -> Resistor_SMD:R_0603_1608Metric
- R10: renamed from R8; value 100K -> 100k; footprint Resistor_SMD:R_0603_1608Metric_Pad0.98x0.95mm_HandSolder -> Resistor_SMD:R_0603_1608Metric; MFG Walsin Technologies -> (none); MPN WR04X1003FTL -> (none); Manufacturer Walsin Technologies -> (none); body_length 1 mm -> (none); case_code_imperial 0402 -> (none); composition Thick Film -> (none); contact_material Tin -> (none); depth 500 µm -> (none); grade 消费级 -> (none); lead_free Lead Free -> (none); military_standard Not -> (none); mount 表面贴装 -> (none); operating_temperature -55 °C -> (none); overload_voltage 50 V -> (none); package 0402 -> (none); packaging Tape and Reel -> (none); power_rating 62.5 mW -> (none); reach_svhc_compliant Unknown -> (none); resistance 100 kΩ -> (none); technology 厚膜 -> (none); temperature_coefficient 100 ppm/°C -> (none); terminal_pitch 0.75 mm -> (none); termination SMD -> (none); tolerance 1 % -> (none); type 厚膜电阻 -> (none); voltage_rating 50 V -> (none)
- R11: renamed from R9; value 22K -> 22.1k; footprint Resistor_SMD:R_0603_1608Metric_Pad0.98x0.95mm_HandSolder -> Resistor_SMD:R_0603_1608Metric; MFG Vishay -> (none); MPN CRCW040222K0FKED -> (none); Manufacturer Vishay -> (none); body_length 1 mm -> (none); body_width 500 µm -> (none); case_code_imperial 0402 -> (none); characteristic Automotive AEC-Q200 -> (none); composition Thick Film -> (none); contact_plating Tin -> (none); depth 500 µm -> (none); height 350 µm -> (none); lead_free Lead Free -> (none); material Thick Film -> (none); military_standard Not -> (none); mount Surface Mount -> (none); number_of_terminations 2 -> (none); operating_temperature -55 °C -> (none); overload_voltage 75 V -> (none); package 0402 -> (none); package_quantity 10 -> (none); packaging Tape and Reel -> (none); power_dissipation 63 mW -> (none); power_rating 62.5 mW -> (none); radiation_hardening No -> (none); reach_svhc_compliant Unknown -> (none); resistance 22 kΩ -> (none); temperature_coefficient 100 ppm/°C -> (none); terminal_pitch 0.75 mm -> (none); termination SMD -> (none); tolerance 1 % -> (none); type 厚膜电阻 -> (none); voltage_rating 50 V -> (none)
- R12: renamed from R7; value 100K -> 0603WAF1003T5E; footprint Resistor_SMD:R_0603_1608Metric_Pad0.98x0.95mm_HandSolder -> Resistor_SMD:R_0603_1608Metric
- R13: renamed from R10; value 1.8M -> RK73H1JTTD1804F
- R4: renamed from R3; footprint Resistor_SMD:R_0603_1608Metric_Pad0.98x0.95mm_HandSolder -> Resistor_SMD:R_0603_1608Metric; now not fitted; now left out of the parts list
- R5: renamed from R4; footprint Resistor_SMD:R_0603_1608Metric_Pad0.98x0.95mm_HandSolder -> Resistor_SMD:R_0603_1608Metric; now not fitted; now left out of the parts list
- R7: renamed from R6; value 1M -> 1MΩ; footprint Resistor_SMD:R_0603_1608Metric_Pad0.98x0.95mm_HandSolder -> Resistor_SMD:R_0603_1608Metric
- R9: renamed from R5; value 10K -> 10k; footprint Resistor_SMD:R_0603_1608Metric_Pad0.98x0.95mm_HandSolder -> Resistor_SMD:R_0603_1608Metric; symbol RC0402JR-0710KL:RC0402JR-0710KL -> Project_Passives:RC0603JR-0710KL_3c0a9a7d; MFG Yageo -> (none); MPN RC0402JR-0710KL -> RC0603JR-0710KL; Manufacturer Yageo -> YAGEO; Power (none) -> 0.1W; Resistance (none) -> 10k; Tolerance (none) -> 5%; body_length 1 mm -> (none); body_width 0.5 mm -> (none); case_code_imperial 0402 -> (none); composition Thick Film -> (none); depth 500 µm -> (none); grade 消费级 -> (none); height 0.016 in -> (none); height_overall 0.35 mm -> (none); lead_free Lead Free -> (none); military_standard Not -> (none); mount SMT -> (none); number_of_terminations 2 -> (none); operating_temperature -55 °C -> (none); overload_voltage 50 V -> (none); package 0402 -> 0603; package_quantity 1 -> (none); packaging Tape and Reel -> (none); pins 2 -> (none); power_dissipation 63 mW -> (none); power_rating 62.5 mW -> (none); reach_svhc_compliant Unknown -> (none); resistance 10 kΩ -> (none); technology 厚膜 -> (none); temperature_coefficient 100 ppm/°C -> (none); terminal_pitch 0.75 mm -> (none); termination SMD -> (none); tolerance 0.05 -> (none); type 厚膜电阻 -> (none); voltage_rating 50 V -> (none)
- U1: footprint Package_SO:SOIC-8_3.9x4.9mm_P1.27mm -> kicad_api_lib:XL1509-5.0
- U2: footprint kicad_api_lib:IB0505S-2W3L -> IB0505S-2W3L:IB0505S-2W3L; now not fitted; now left out of the parts list
- U3: input_voltage 3 V, 5.5 V -> 2.5 V to 5.5 V; output_voltage 5.5 V, 600 mV -> 3.315 V nominal; now not fitted; now left out of the parts list
- U4: now not fitted; now left out of the parts list
- U5: renamed from U18; fet_type (none) -> P通道; huaqiu_pn (none) -> G4607254; lead_free (none) -> Yes; mount (none) -> SMT; package (none) -> SC-70-6; packaging (none) -> 3000pcs; voltage (none) -> 1.5 V
- U6: renamed from U5; value SY8089AAC -> SY8089A1AAC; footprint Package_TO_SOT_SMD:SOT-23-5_HandSoldering -> Package_TO_SOT_SMD:SOT-23-5; symbol SY8089AAC:SY8089AAC -> Project_Power:SY8089A1AAC; MPN SY8089AAC -> SY8089A1AAC
- renumbered C58 to C9, D4 to D5, L2 to L1
Connections:
- net +24V: now also R3.1; no longer D7.1 (K), Q1.1 (S), Q1.2 (S), Q1.3 (S), Q2.1 (E)
- net +3V3: now also D3.2 (A); no longer D2.2 (A)
- net +5V: now also D2.2 (A); no longer D3.2 (A)
- net Earth: now also C10.2, C12.2, R6.2, R8.2
- net GND: now also C10.1, C12.1, D4.1 (K), R6.1, R8.1
- net +3V3_ISO renamed +3V3S
- net +5V_ISO renamed +5VS
- net VBUS renamed +1V8
- net +1V8: now also D7.1 (K), Q1.1 (S), Q1.2 (S), Q1.3 (S), Q2.1 (E)
- new net: D4.2 (A), R3.2
Other:
- note added: "CN1：24 V 电源输入；D1：输入瞬态钳位。 U1 / D5 / L1 / C5：降压与输出滤波。 输出网络为 BOARD_5V_RAW，送 PWR-02。"
- note added: "D2：+5V；D3：+3V3；D4：+24V。 R1~R3 为限流电阻；LED 均为 0603。"
- note added: "H1~H4：连接金属安装板；R6~R8 与 C10~C12 提供泄放 / 高频耦合。USB 页另有 FB2 / C60。"
- note added: "PWR-01 24 V 输入与 5 V 降压"
- note added: "PWR-02 板内 5 V 防倒灌支路"
- note added: "PWR-03 +5V 转 +3V3"
- note added: "PWR-04 电源状态指示"
- note added: "PWR-05 Earth / GND 与安装孔"
- note added: "PWR-06 隔离供电与稳压预留【备用 / DNP】"
- note added: "PWR-07 MOS 电源保护预留【备用 / DNP】"
- note added: "Q1 / Q2 / D6 / D7：原电源保护备用方案。 当前不在已装配供电路径中，不能视为现有输入保护。 该分区仅标识用途，启用前需独立复核。"
- note added: "U2：隔离 DC-DC；U4 / U3：后级稳压。 +5VS / +3V3S / GNDS 为备用电源域。 当前相关元件不装配，启用前复核参数。"
- note added: "U5：BOARD_5V_RAW → +5V。 与 USB 的两路 LM66100 支路汇合至 +5V。 C9、C13：输入与输出旁路。"
- note added: "U6 / L3：+3V3 稳压，供 MCU 与逻辑接口。 R10 / R11：反馈分压；C14 / C17 / C18：滤波去耦。"
- note added: "装配说明：实线框内按元件属性装配；虚线框为保留方案。 22 µF / 0603 电容需按工作电压核对有效容量；以上分区不改变现有元件参数。"
- note removed: "Input Anti-Reverse & Backflow Protection Circuit"
- note removed: "SY8089AAC_DCDC Module"
- note removed: "VOUT = 0.6 * (1+R2/R3)"
- note removed: "XL1509-5.0_DCDC Module"
- note removed: "模块电路功能： 该原理图功能是对输入电源进行防反接以及过流保护"
- note removed: "模块电路功能： 输入2.7V-5.5V，输出3.3V，可提供 2A 连续电流和 3A 峰值电流"
- note removed: "模块电路功能： 这是一个高效的同步降压DC-DC转换器电路， 核心功能是将4.5V-40V范围的直流输入降压为稳定的5V直流输出， 最大带载能力为2A。 供电电压： VIN：4.5V-40V； +5V：固定输出； 应用场景： 嵌入式/单片机系统供电：（为传感器、无线模块、接口外设提供稳定 5V 工作电源）、 网络通信设备辅电：（交换机、路由器、光猫、POE 终端设备内部的 5V 辅助电源）、 消费电子内部供电：（机顶盒、硬盘盒、桌面显示设备的 5V 系统电源）等。"
- moved on the sheet: C1, C11, C13, C14, C15, C16, C17, C18, C19, C5, C9, CN1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
