File: POWER.kicad_sch (KiCad schematic)
At the start: 55 parts, among them CN1 KF128L-5.08-2P, Q1 AP40P04Q, Q2 MMDT5401, U1 XL1509-5.0, U2 IB0505S-2W3L, U3 SY8089A1AAC, U4 CH213K, U5 LM66100DCKR, U6 SY8089A1AAC

Commit message: V2.0: update motor control schematics, replicated PCB layout and component libraries
Save current KiCad design progress, including four motor control layouts and new component libraries. PCB routing and DRC cleanup remain unfinished; this is not a fabrication release.
Parts:
- CN1: value KF128L-5.08-2P -> KF2EDGK-5.08-2P; footprint kicad_api_lib:KF128L-5.08-2P -> kicad_api_lib:KF2EDGR-5.08-2P; symbol KF128L-5.08-2P:15ETYRC-3.5-02P-14-00AH -> KF2EDGK-5.08-2P:KF2EDGK-5.08-2P; Footprint_Source (none) -> KEFA KF2EDGR-5.08 Rev B 2024-09-26; verify purchased part d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; MPN KF128L-5.08-2P -> KF2EDGR-5.08-2P; Manufacturer KEFA -> (none); Mating_Plug (none) -> KF2EDGK-5.08-2P; current 10 A, 24 A -> (none); current_rating 24 A -> (none); huaqiu_pn G3175735 -> (none); mount 直针 -> 弯针板座 + 可插拔接线端子; operating_temperature -40 °C -> (none); package 插件,P=5.08mm -> THT, P=5.08mm, drill=1.6mm; termination_type 螺钉 -> (none); voltage 250 V, 300 V -> (none); voltage_rating 250 V -> (none); wire_gauge 2.5 -> (none)
Connections:
- net +24V: now also D4.2 (A); no longer R3.1
- net GND: now also R3.2; no longer D4.1 (K)
- new net: D4.1 (K), R3.1
Other:
- moved on the sheet: R3
Changed lines of the file:
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@@
 	(wire
 		(pts
+			(xy 81.28 155.194) (xy 81.28 157.988)
+		)
+		(stroke
+			(width 0)
+			(type default)
+		)
+	)
+	(wire
+		(pts
 			(xy 182.245 180.34) (xy 191.135 180.34)
 		)
@@
 	(wire
 		(pts
+			(xy 81.28 165.608) (xy 81.28 167.64)
+		)
+		(stroke
+			(width 0)
+			(type default)
+		)
+	)
+	(wire
+		(pts
 			(xy 90.17 219.71) (xy 90.17 222.25)
 		)
@@
 	(wire
 		(pts
-			(xy 81.28 183.134) (xy 81.28 177.038)
-		)
-		(stroke
-			(width 0)
-			(type default)
-		)
-	)
-	(wire
-		(pts
 			(xy 82.55 69.85) (xy 82.55 81.28)
 		)
@@
 	(wire
 		(pts
-			(xy 81.28 169.418) (xy 81.28 166.116)
-		)
-		(stroke
-			(width 0)
-			(type default)
-		)
-	)
-	(wire
-		(pts
 			(xy 518.16 173.99) (xy 518.16 177.8)
 		)
@@
 	(wire
 		(pts
-			(xy 81.28 155.194) (xy 81.28 158.496)
-		)
-		(stroke
-			(width 0)
-			(type default)
-		)
-	)
-	(wire
-		(pts
 			(xy 333.375 44.45) (xy 329.565 44.45)
 		)
@@
 	(wire
 		(pts
+			(xy 81.28 175.26) (xy 81.28 183.134)
+		)
+		(stroke
+			(width 0)
+			(type default)
+		)
+	)
+	(wire
+		(pts
 			(xy 495.3 219.71) (xy 510.54 219.71)
 		)
@@
 	)
 	(symbol
+		(lib_id "Device:LED")
+		(at 81.28 161.798 90)
+		(unit 1)
+		(body_style 1)
+		(exclude_from_sim no)
+		(in_bom yes)
+		(on_board yes)
+		(in_pos_files yes)
+		(dnp no)
+		(fields_autoplaced yes)
+		(property "Reference" "D4"
+			(at 85.09 162.1154 90)
+			(show_name no)
+			(do_not_autoplace no)
+			(effects
+				(font
+					(size 1.27 1.27)
+				)
+				(justify right)
+			)
+		)
+		(property "Value" "LED"
+			(at 85.09 164.6554 90)
+			(show_name no)
+			(do_not_autoplace no)
+			(effects
+				(font
+					(size 1.27 1.27)
+				)
+				(justify right)
+			)
+		)
+		(property "Footprint" "LED_SMD:LED_0603_1608Metric"
+			(at 81.28 161.798 0)
+			(hide yes)
+			(show_name no)
+			(do_not_autoplace no)
+			(effects
+				(font
+					(size 1.27 1.27)
+				)
+			)
+		)
+		(property "Datasheet" ""
+			(at 81.28 161.798 0)
+			(hide yes)
+			(show_name no)
+			(do_not_autoplace no)
+			(effects
+				(font
+					(size 1.27 1.27)
+				)
+			)
+		)
+		(property "Description" "Light emitting diode"
+			(at 81.28 161.798 0)
+			(hide yes)
+			(show_name no)
+			(do_not_autoplace no)
+			(effects
+				(font
+					(size 1.27 1.27)
+				)
+			)
+		)
+		(property "Sim.Pins" "1=K 2=A"
+			(at 81.28 161.798 0)
+			(hide yes)
+			(show_name no)
+			(do_not_autoplace no)
+			(effects
+				(font
+					(size 1.27 1.27)
+				)
+			)
+		)
+		(pin "2"
+		)
+		(pin "1"
+		)
+		(instances
+			(project "GD32F303VET6_4Motor_Control"
+				(path "/54005433-e3aa-4693-8f75-bb73943288d3/991ba235-e77c-4edd-a3a2-0f8fb1340e9c"
+					(reference "D4")
+					(unit 1)
+				)
+			)
+		)
+	)
+	(symbol
 		(lib_id "Device:C")
 		(at 81.28 218.44 0)
@@
 	)
 	(symbol
-		(lib_id "KF128L-5.08-2P:15ETYRC-3.5-02P-14-00AH")
+		(lib_id "KF2EDGK-5.08-2P:KF2EDGK-5.08-2P")
 		(at 55.88 45.085 180)
 		(unit 1)
@@
 			)
 		)
-		(property "Value" "KF128L-5.08-2P"
+		(property "Value" "KF2EDGK-5.08-2P"
 			(at 55.88 50.3427 0)
 			(show_name no)
@@
 			)
 		)
-		(property "Footprint" "kicad_api_lib:KF128L-5.08-2P"
+		(property "Footprint" "kicad_api_lib:KF2EDGR-5.08-2P"
 			(at 55.88 48.895 0)
 			(hide yes)
@@
 			)
 		)
-		(property "Datasheet" "http://file.elecfans.com/web1/M00/E3/BD/pIYBAGBBnUaAMkBFAAMGNHK6UP8913.pdf"
+		(property "Datasheet" "https://a0.ldycdn.com/KF2EDGR-5.08-aidqoBpqKirRlkSlqrkpklpj.pdf"
 			(at 55.88 48.895 0)
 			(hide yes)
@@
 			)
 		)
-		(property "Description" "间距:5.08mm;结构:1x2P;排数:1;每排PIN数:2;安装方式:直针;额定电流:24A;额定电压:250V;线规 - AWG:12~22;线规 - mm2:2.5;工作温度范围:-40℃~+105℃;颜色:绿色;"
+		(property "Description" "5.08mm 2P pluggable terminal set: KF2EDGK cable plug + KF2EDGR right-angle PCB header; PCB footprint follows KEFA header drawing; verify purchased mating pair."
 			(at 55.88 48.895 0)
 			(hide yes)
@@
 			)
 		)
-		(property "MPN" "KF128L-5.08-2P"
+		(property "MPN" "KF2EDGR-5.08-2P"
 			(at 55.88 45.085 0)
 			(hide yes)
@@
 			)
 		)
-		(property "Manufacturer" "KEFA"
+		(property "Manufacturer" ""
 			(at 55.88 45.085 0)
 			(hide yes)
@@
 			)
 		)
-		(property "current" "10 A, 24 A"
-			(at 55.88 45.085 0)
-			(hide yes)
-			(show_name no)
-			(do_not_autoplace no)
-			(effects
-				(font
-					(size 1.27 1.27)
-				)
-			)
-		)
-		(property "current_rating" "24 A"
-			(at 55.88 45.085 0)
-			(hide yes)
-			(show_name no)
-			(do_not_autoplace no)
-			(effects
-				(font
-					(size 1.27 1.27)
-				)
-			)
-		)
-		(property "huaqiu_pn" "G3175735"
-			(at 55.88 45.085 0)
-			(hide yes)
-			(show_name no)
-			(do_not_autoplace no)
-			(effects
-				(font
-					(size 1.27 1.27)
-				)
-			)
-		)
-		(property "mount" "直针"
+		(property "mount" "弯针板座 + 可插拔接线端子"
 			(at 55.88 45.085 0)
 			(hide yes)
@@
 			)
 		)
-		(property "operating_temperature" "-40 °C"
-			(at 55.88 45.085 0)
-			(hide yes)
-			(show_name no)
-			(do_not_autoplace no)
-			(effects
-				(font
-					(size 1.27 1.27)
-				)
-			)
-		)
-		(property "package" "插件,P=5.08mm"
+		(property "package" "THT, P=5.08mm, drill=1.6mm"
 			(at 55.88 45.085 0)
 			(hide yes)
@@
 			)
 		)
-		(property "termination_type" "螺钉"
+		(property "Mating_Plug" "KF2EDGK-5.08-2P"
 			(at 55.88 45.085 0)
 			(hide yes)
@@
 			)
 		)
-		(property "voltage" "250 V, 300 V"
-			(at 55.88 45.085 0)
-			(hide yes)
-			(show_name no)
-			(do_not_autoplace no)
-			(effects
-				(font
-					(size 1.27 1.27)
-				)
-			)
-		)
-		(property "voltage_rating" "250 V"
-			(at 55.88 45.085 0)
-			(hide yes)
-			(show_name no)
-			(do_not_autoplace no)
-			(effects
-				(font
-					(size 1.27 1.27)
-				)
-			)
-		)
-		(property "wire_gauge" "2.5"
+		(property "Footprint_Source" "KEFA KF2EDGR-5.08 Rev B 2024-09-26; verify purchased part dimensions"
 			(at 55.88 45.085 0)
 			(hide yes)
@@
 	(symbol
 		(lib_id "Device:R_US")
-		(at 81.28 162.306 0)
+		(at 81.28 171.45 0)
 		(unit 1)
 		(body_style 1)
@@
 		(fields_autoplaced yes)
 		(property "Reference" "R3"
-			(at 83.82 161.0359 0)
+			(at 83.82 170.1799 0)
 			(show_name no)
 			(do_not_autoplace no)
@@
 		)
 		(property "Value" "10kΩ"
-			(at 83.82 163.5759 0)
+			(at 83.82 172.7199 0)
 			(show_name no)
 			(do_not_autoplace no)
@@
 		)
 		(property "Footprint" "Resistor_SMD:R_0603_1608Metric"
-			(at 82.296 162.56 90)
+			(at 82.296 171.704 90)
 			(hide yes)
 			(show_name no)
@@
 		)
 		(property "Datasheet" ""
-			(at 81.28 162.306 0)
+			(at 81.28 171.45 0)
 			(hide yes)
 			(show_name no)
@@
 		)
 		(property "Description" "Resistor, US symbol"
-			(at 81.28 162.306 0)
+			(at 81.28 171.45 0)
 			(hide yes)
 			(show_name no)
@@
 					(unit 1)
 				)
-			)
-		)
-	)
-	(symbol
-		(lib_id "Device:LED")
-		(at 81.28 173.228 90)
-		(unit 1)
-		(body_style 1)
-		(exclude_from_sim no)
-		(in_bom yes)
-		(on_board yes)
-		(in_pos_files yes)
-		(dnp no)
-		(fields_autoplaced yes)
-		(property "Reference" "D4"
-			(at 85.09 173.5454 90)
-			(show_name no)
-			(do_not_autoplace no)
-			(effects
-				(font
-					(size 1.27 1.27)
-				)
-				(justify right)
-			)
-		)
-		(property "Value" "LED"
-			(at 85.09 176.0854 90)
-			(show_name no)
-			(do_not_autoplace no)
-			(effects
-				(font
-					(size 1.27 1.27)
-				)
-				(justify right)
-			)
-		)
-		(property "Footprint" "LED_SMD:LED_0603_1608Metric"
-			(at 81.28 173.228 0)
-			(hide yes)
-			(show_name no)
-			(do_not_autoplace no)
-			(effects
-				(font
-					(size 1.27 1.27)
-				)
-			)
-		)
-		(property "Datasheet" ""
-			(at 81.28 173.228 0)
-			(hide yes)
-			(show_name no)
-			(do_not_autoplace no)
-			(effects
-				(font
-					(size 1.27 1.27)
-				)
-			)
-		)
-		(property "Description" "Light emitting diode"
-			(at 81.28 173.228 0)
-			(hide yes)
-			(show_name no)
-			(do_not_autoplace no)
-			(effects
-				(font
-					(size 1.27 1.27)
-				)
-			)
-		)
-		(property "Sim.Pins" "1=K 2=A"
-			(at 81.28 173.228 0)
-			(hide yes)
-			(show_name no)
-			(do_not_autoplace no)
-			(effects
-				(font
-					(size 1.27 1.27)
-				)
-			)
-		)
-		(pin "2"
-		)
-		(pin "1"
-		)
-		(instances
-			(project "GD32F303VET6_4Motor_Control"
-				(path "/54005433-e3aa-4693-8f75-bb73943288d3/991ba235-e77c-4edd-a3a2-0f8fb1340e9c"
-					(reference "D4")
-					(unit 1)
-				)

Commit message: 更新V2.0电路设计及0.5oz内层制造交付资料
Parts:
- added TP_24V1: 24V, kicad_api_lib:TestPoint_Pad_D1.143mm, symbol Connector:TestPoint
- added TP_3V3: 3V3, kicad_api_lib:TestPoint_Pad_D1.143mm, symbol Connector:TestPoint
- added TP_5V1: 5V, kicad_api_lib:TestPoint_Pad_D1.143mm, symbol Connector:TestPoint
- added TP_5V_RAW1: 5V_RAW, kicad_api_lib:TestPoint_Pad_D1.143mm, symbol Connector:TestPoint
- added TP_GND_PWR1: GND_PWR, kicad_api_lib:TestPoint_Pad_D1.016mm, symbol Connector:TestPoint
- H1, H2, H3, H4: footprint (none) -> MountingHole:MountingHole_3.2mm_M3_ISO7380_Pad
Connections:
- net +24V: now also TP_24V1.1
- net +3V3: now also TP_3V3.1
- net +5V: now also TP_5V1.1
- net BOARD_5V_RAW: now also TP_5V_RAW1.1
- net GND: now also TP_GND_PWR1.1
Other:
- note added: "CN1：24V 输入；D1：输入瞬态钳位。 U1 / D5 / L1 / C5：降压及输出滤波。 BOARD_5V_RAW 送至 PWR-02。"
- note added: "D2：+5V；D3：+3V3；D4：+24V。 R1～R3 限流；仅表示对应电源电压。"
- note added: "H1～H4 接 Earth 金属安装板。 R6～R8 / C10～C12：泄放与高频耦合。"
- note added: "POWER TEST POINTS"
- note added: "PWR-01 24V 输入与 5V 降压"
- note added: "PWR-02 板内 5V 防倒灌"
- note added: "PWR-03 5V 转 3.3V"
- note added: "PWR-04 供电状态指示"
- note added: "PWR-05 机壳耦合与安装孔"
- note added: "PWR-06 隔离供电预留【DNP】"
- note added: "PWR-07 MOS 电源保护预留【DNP】"
- note added: "Q1 / Q2 / D6 / D7：保留的电源保护方案。 当前不装配，不构成现有供电保护路径。"
- note added: "U2：隔离 DC-DC；U3 / U4：后级稳压。 +5VS / +3V3S / GNDS 为备用电源域。"
- note added: "U5：LM66100，接入 +5V 汇流。 C9 / C13：输入、输出旁路。 与 USB 的 U24 / U25 支路汇合。"
- note added: "U6 / L3：3.3V 稳压；R10 / R11：反馈。 C14～C18：输入、输出及反馈滤波。"
- note added: "备用区保留原接线；启用前需独立复核。电容有效容量需结合偏压与具体料号校核。"
- note removed: "CN1：24 V 电源输入；D1：输入瞬态钳位。 U1 / D5 / L1 / C5：降压与输出滤波。 输出网络为 BOARD_5V_RAW，送 PWR-02。"
- note removed: "D2：+5V；D3：+3V3；D4：+24V。 R1~R3 为限流电阻；LED 均为 0603。"
- note removed: "H1~H4：连接金属安装板；R6~R8 与 C10~C12 提供泄放 / 高频耦合。USB 页另有 FB2 / C60。"
- note removed: "PWR-01 24 V 输入与 5 V 降压"
- note removed: "PWR-02 板内 5 V 防倒灌支路"
- note removed: "PWR-03 +5V 转 +3V3"
- note removed: "PWR-04 电源状态指示"
- note removed: "PWR-05 Earth / GND 与安装孔"
- note removed: "PWR-06 隔离供电与稳压预留【备用 / DNP】"
- note removed: "PWR-07 MOS 电源保护预留【备用 / DNP】"
- note removed: "Q1 / Q2 / D6 / D7：原电源保护备用方案。 当前不在已装配供电路径中，不能视为现有输入保护。 该分区仅标识用途，启用前需独立复核。"
- note removed: "U2：隔离 DC-DC；U4 / U3：后级稳压。 +5VS / +3V3S / GNDS 为备用电源域。 当前相关元件不装配，启用前复核参数。"
- note removed: "U5：BOARD_5V_RAW → +5V。 与 USB 的两路 LM66100 支路汇合至 +5V。 C9、C13：输入与输出旁路。"
- note removed: "U6 / L3：+3V3 稳压，供 MCU 与逻辑接口。 R10 / R11：反馈分压；C14 / C17 / C18：滤波去耦。"
- note removed: "装配说明：实线框内按元件属性装配；虚线框为保留方案。 22 µF / 0603 电容需按工作电压核对有效容量；以上分区不改变现有元件参数。"
