File: RS232.kicad_sch (KiCad schematic)
At the start: 10 parts, among them CN3 WJ15EDGRC-3.81-2P, U10 SP3232EEN-L/TR

Commit message: 更新V2.0电路设计及0.5oz内层制造交付资料
Other:
- note added: "232-01 收发器 / 电荷泵 / 滤波【DNP】"
- note added: "232-02 对外接口【DNP】"
- note added: "232-03 功能与装配说明【DNP】"
- note added: "U10：SP3232 电平转换；C43 / C44 / C46 / C47：电荷泵；C45：去耦。 R22 / R23 / FB1：串联阻抗与滤波；CN3 引出 RS232 两路信号。 MCU 端接 PC10 / PC11；本页全部 DNP，启用前核对外设选择与收发方向。"
- note removed: "232-01 收发器 / 电荷泵 / 滤波【备用 / DNP】"
- note removed: "232-01：U10 将 MCU UART 与 RS232 电平互相转换。 C43 / C44 / C46 / C47 为电荷泵相关电容；C45 为电源去耦。 R22 / R23 / FB1 为串联阻抗及滤波。 232-02：CN3 引出 RS232_TX1、RS232_RX1，外接设备需具备共同参考地。 本页器件当前均为 DNP；启用前复核 MCU TX / RX 的实际收发方向与接线。"
- note removed: "232-02 对外串口【备用 / DNP】"
Changed lines of the file:
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@@
 	(paper "A4")
+	(rectangle
+		(start 219 62)
+		(end 279 124)
+		(stroke
+			(width 0.254)
+			(type dash)
+		)
+		(fill
+			(type none)
+		)
+	)
+	(rectangle
+		(start 23 133)
+		(end 279 163)
+		(stroke
+			(width 0.254)
+			(type dash)
+		)
+		(fill
+			(type none)
+		)
+	)
 	(rectangle
 		(start 80 62)
@@
 		)
 	)
-	(rectangle
-		(start 219 62)
-		(end 279 124)
-		(stroke
-			(width 0.254)
-			(type dash)
+	(text "232-03  功能与装配说明【DNP】"
+		(exclude_from_sim no)
+		(at 26 136 0)
+		(effects
+			(font
+				(face "Microsoft YaHei")
+				(size 2 2)
+				(bold yes)
+			)
+			(justify left top)
 		)
-		(fill
-			(type none)
+	)
+	(text "232-01  收发器 / 电荷泵 / 滤波【DNP】"
+		(exclude_from_sim no)
+		(at 83 65 0)
+		(effects
+			(font
+				(face "Microsoft YaHei")
+				(size 2 2)
+				(bold yes)
+			)
+			(justify left top)
+		)
+	)
+	(text "U10：SP3232 电平转换；C43 / C44 / C46 / C47：电荷泵；C45：去耦。\nR22 / R23 / FB1：串联阻抗与滤波；CN3 引出 RS232 两路信号。\nMCU 端接 PC10 / PC11；本页全部 DNP，启用前核对外设选择与收发方向。"
+		(exclude_from_sim no)
+		(at 28 146 0)
+		(effects
+			(font
+				(face "Microsoft YaHei")
+				(size 1.7 1.7)
+			)
+			(justify left top)
+		)
+	)
+	(text "232-02  对外接口【DNP】"
+		(exclude_from_sim no)
+		(at 222 65 0)
+		(effects
+			(font
+				(face "Microsoft YaHei")
+				(size 2 2)
+				(bold yes)
+			)
+			(justify left top)
 		)
 	)
@@
 		(effects
 			(font
-				(face "宋体")
+				(face "Microsoft YaHei")
 				(size 3 3)
 			)
 			(justify left top)
-		)
-	)
-	(text "232-01：U10 将 MCU UART 与 RS232 电平互相转换。\nC43 / C44 / C46 / C47 为电荷泵相关电容；C45 为电源去耦。\nR22 / R23 / FB1 为串联阻抗及滤波。\n232-02：CN3 引出 RS232_TX1、RS232_RX1，外接设备需具备共同参考地。\n\n本页器件当前均为 DNP；启用前复核 MCU TX / RX 的实际收发方向与接线。"
-		(exclude_from_sim no)
-		(at 24 137 0)
-		(effects
-			(font
-				(face "宋体")
-				(size 1.8 1.8)
-			)
-			(justify left top)
-		)
-	)
-	(text "232-02  对外串口【备用 / DNP】"
-		(exclude_from_sim no)
-		(at 222 65 0)
-		(effects
-			(font
-				(face "宋体")
-				(size 1.8 1.8)
-				(bold yes)
-			)
-			(justify left top)
-		)
-	)
-	(text "232-01  收发器 / 电荷泵 / 滤波【备用 / DNP】"
-		(exclude_from_sim no)
-		(at 83 65 0)
-		(effects
-			(font
-				(face "宋体")
-				(size 1.8 1.8)
-				(bold yes)
-			)
-			(justify left top)
