File: WiFi_OTA.kicad_sch (KiCad schematic)
At the start: 15 parts, among them J3 TYPE-C-31-M-31, SW2 RESET, SW3 BOOT, U26 ESP32-C3-WROOM-02-N4

Commit message: 停用 WiFi OTA 装配并从 PCB 排除
Parts:
- C68, C69, C70, J3, R79, R80, R81, R82, R87, R88, R89, R90, SW2, SW3, U26: now not fitted; now left out of the parts list
Changed lines of the file:
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@@
 		(body_style 1)
 		(exclude_from_sim no)
-		(in_bom yes)
-		(on_board yes)
-		(in_pos_files yes)
-		(dnp no)
+		(in_bom no)
+		(on_board no)
+		(in_pos_files yes)
+		(dnp yes)
 		(property "Reference" "R80"
 			(at 314.96 46.99 0)
@@
 		(body_style 1)
 		(exclude_from_sim no)
-		(in_bom yes)
-		(on_board yes)
-		(in_pos_files yes)
-		(dnp no)
+		(in_bom no)
+		(on_board no)
+		(in_pos_files yes)
+		(dnp yes)
 		(property "Reference" "J3"
 			(at 71.12 170.18 0)
@@
 		(body_style 1)
 		(exclude_from_sim no)
-		(in_bom yes)
-		(on_board yes)
-		(in_pos_files yes)
-		(dnp no)
+		(in_bom no)
+		(on_board no)
+		(in_pos_files yes)
+		(dnp yes)
 		(property "Reference" "R90"
 			(at 294.64 205.74 90)
@@
 		(body_style 1)
 		(exclude_from_sim no)
-		(in_bom yes)
-		(on_board yes)
-		(in_pos_files yes)
-		(dnp no)
+		(in_bom no)
+		(on_board no)
+		(in_pos_files yes)
+		(dnp yes)
 		(property "Reference" "C70"
 			(at 193.04 102.87 0)
@@
 		(body_style 1)
 		(exclude_from_sim no)
-		(in_bom yes)
-		(on_board yes)
-		(in_pos_files yes)
-		(dnp no)
+		(in_bom no)
+		(on_board no)
+		(in_pos_files yes)
+		(dnp yes)
 		(property "Reference" "R87"
 			(at 58.42 250.19 0)
@@
 		(body_style 1)
 		(exclude_from_sim no)
-		(in_bom yes)
-		(on_board yes)
-		(in_pos_files yes)
-		(dnp no)
+		(in_bom no)
+		(on_board no)
+		(in_pos_files yes)
+		(dnp yes)
 		(property "Reference" "SW2"
 			(at 266.7 102.87 0)
@@
 		(body_style 1)
 		(exclude_from_sim no)
-		(in_bom yes)
-		(on_board yes)
-		(in_pos_files yes)
-		(dnp no)
+		(in_bom no)
+		(on_board no)
+		(in_pos_files yes)
+		(dnp yes)
 		(property "Reference" "R82"
 			(at 386.08 46.99 0)
@@
 		(body_style 1)
 		(exclude_from_sim no)
-		(in_bom yes)
-		(on_board yes)
-		(in_pos_files yes)
-		(dnp no)
+		(in_bom no)
+		(on_board no)
+		(in_pos_files yes)
+		(dnp yes)
 		(property "Reference" "SW3"
 			(at 355.6 92.71 0)
@@
 		(body_style 1)
 		(exclude_from_sim no)
-		(in_bom yes)
-		(on_board yes)
-		(in_pos_files yes)
-		(dnp no)
+		(in_bom no)
+		(on_board no)
+		(in_pos_files yes)
+		(dnp yes)
 		(property "Reference" "R79"
 			(at 193.04 85.09 0)
@@
 		(body_style 1)
 		(exclude_from_sim no)
-		(in_bom yes)
-		(on_board yes)
-		(in_pos_files yes)
-		(dnp no)
+		(in_bom no)
+		(on_board no)
+		(in_pos_files yes)
+		(dnp yes)
 		(fields_autoplaced yes)
 		(property "Reference" "U26"
@@
 		(body_style 1)
 		(exclude_from_sim no)
-		(in_bom yes)
-		(on_board yes)
-		(in_pos_files yes)
-		(dnp no)
+		(in_bom no)
+		(on_board no)
+		(in_pos_files yes)
+		(dnp yes)
 		(property "Reference" "R81"
 			(at 350.52 46.99 0)
@@
 		(body_style 1)
 		(exclude_from_sim no)
-		(in_bom yes)
-		(on_board yes)
-		(in_pos_files yes)
-		(dnp no)
+		(in_bom no)
+		(on_board no)
+		(in_pos_files yes)
+		(dnp yes)
 		(property "Reference" "R88"
 			(at 109.22 250.19 0)
@@
 		(body_style 1)
 		(exclude_from_sim no)
-		(in_bom yes)
-		(on_board yes)
-		(in_pos_files yes)
-		(dnp no)
+		(in_bom no)
+		(on_board no)
+		(in_pos_files yes)
+		(dnp yes)
 		(property "Reference" "C68"
 			(at 193.04 46.99 0)
@@
 		(body_style 1)
 		(exclude_from_sim no)
-		(in_bom yes)
-		(on_board yes)
-		(in_pos_files yes)
-		(dnp no)
+		(in_bom no)
+		(on_board no)
+		(in_pos_files yes)
+		(dnp yes)
 		(property "Reference" "R89"
 			(at 294.64 182.88 90)
@@
 		(body_style 1)
 		(exclude_from_sim no)
-		(in_bom yes)
-		(on_board yes)
-		(in_pos_files yes)
-		(dnp no)
+		(in_bom no)
+		(on_board no)
+		(in_pos_files yes)
+		(dnp yes)
 		(property "Reference" "C69"
 			(at 231.14 46.99 0)

Commit message: 更新V2.0电路设计及0.5oz内层制造交付资料
Parts:
- renumbered C70 to C69, C69 to C70, R87 to R66, R88 to R67, R79 to R68, R89 to R69, R90 to R70, R80 to R71, R81 to R72, R82 to R73
Other:
- note added: "C68=10uF、C70=100nF：3V3 去耦。 R68=10k、C69=1uF：EN 延时。 SW2：复位 ESP；沿用板上 +3V3。"
- note added: "R66 / R67：CC1 / CC2 各 5.1k 下拉。 R69 / R70：USB 串联 22Ω，靠近模块。 D+ → GPIO19 / 14；D- → GPIO18 / 13。 VBUS 未接，使用时须由板卡供电。 当前无外置 USB ESD；本页全部不装配。"
- note added: "R71 / R72 / R73：各 10k 启动上拉。 正常 GPIO9 高；下载时拉低。 按住 BOOT → 按放 RESET → 松开 BOOT。"
- note added: "U26：ESP32-C3-WROOM-02-N4。 GPIO4 / 3 脚 TX → GD32 PA10 / 69 RX。 GD32 PA9 / 68 TX → GPIO5 / 4 脚 RX。 GD32 使用 USART0；UART 为 3.3V 直连。 GPIO10 当前未接，不控制 GD32 NRST。 9 / 19 脚接地；其余不用引脚保留 NC。"
- note added: "WIFI-01 ESP32 与 GD32 通信【DNP】"
- note added: "WIFI-02 供电 / EN / RESET【DNP】"
- note added: "WIFI-03 启动配置 / BOOT【DNP】"
- note added: "WIFI-04 原生 USB 下载接口【DNP】"
- note added: "备用页：原理图保留，元件排除 PCB / BOM。 OTA/IAP 规划：网络 → ESP → UART → GD32 / U8 → Bootloader；升级固件尚未实现。"
- note removed: "GPIO4/3 脚 TX → GD32 PD9/56 RX。 GD32 PD8/55 TX → GPIO5/4 脚 RX；UART 直连。 GPIO10/10 脚 → GD32 NRST，双方共用板上 3V3。 GPIO10 必须开漏：拉低复位，高阻释放；禁止推挽高。 与旧 MOS 方案相比，复位命令极性已反转。 未用 GPIO 标 NC；9/19 脚接地。"
- note removed: "OTA/IAP：HTTPS → ESP → UART → GD32/U8 → Bootloader。固件待实现；GPIO10 复位改为低有效。"
- note removed: "R80/R81/R82 = 10k，确保启动电平。 正常：GPIO9 高；下载：GPIO9 低。 按住 BOOT → 按放 RESET → 释放 BOOT。 不加 LED，避免给启动脚增加负载。"
- note removed: "R87/R88：CC1/CC2 各自 5.1k 下拉，不可短接。 R89/R90：22R，靠近模块；USB 差分线短、无长支线。 D+ 接 GPIO19/14 脚，D- 接 GPIO18/13 脚。 VBUS 未接；先给板卡上电，再接 Type-C 数据线。 精简版无外置 USB ESD 保护；保留 BOOT/RESET 恢复。"
- note removed: "WIFI-01 WROOM-02-N4 与 GD32 通信"
- note removed: "WIFI-02 电源 / EN / RESET"
- note removed: "WIFI-03 启动上拉 / BOOT"
- note removed: "WIFI-04 原生 Type-C USB / 最简下载接口"
- note removed: "沿用板上 3V3，不另加 AMS1117。 C68=10uF，C69=100nF 靠近模块。 EN：R79=10k 上拉，C70=1uF 延时。"
